File: duet_pi.kicad_pcb (KiCad board)
At the start: 2 copper layers, 134 x 140 mm, 119 parts, among them J1 Conn_01x03, J10 690-019-298-412, J11 USB_OTG, J13 690-008-221-904, J14 Conn_02x05_Odd_Even, J15 Conn_01x22_Female, J16 Conn_01x22_Female, J17 Molex 470531000, J19 Barrel_Jack, J2 Conn_02x07_Odd_Even, J22 690-019-298-412, J3 Conn_01x03, J4 Conn_01x22_Female, J5 Conn_01x22_Female, J6 THD-02-R, J7 Micro_SD_Card_Det, J8 THD-20-R, J9 THD-02-R, Q1 DMP3013SFV-7, U1 TPD4EUSB30, U11 EMC2301-1-ACZL-TR, U12 RT9742SNGV, U13 FSUSB42MUX, U14 74LVC1G07SE-7, U16 AP64501SP-13, U18 RT9742GGJ5, U2 TPD4EUSB30, U3 MagJack-A70-112-331N126, U4 TPD4EUSB30, U5 74LVC1G07SE-7, U6 USB2514B-I/M2, U7 AP22653W6, U8 PCF85063AT/AAZ, U9 74LVC1G07SE-7, Y1 24MHz, Y2 X32K768S301

Commit message: CM5
Parts:
- removed BT1: Battery_Cell, Battery:BatteryHolder_Keystone_3034_1x20mm
- removed C1, C11, C12, C13, C14, C15, C22, C23, C24, C3, C4, C40, C46, C57, C58, C7: 100n, Capacitor_SMD:C_0402_1005Metric
- removed C10, C17, C19, C2, C20, C21, C47, C49, C5, C51, C52, C6: 10u, Capacitor_SMD:C_0805_2012Metric
- removed C16, C18: 100uF, Capacitor_Tantalum_SMD:CP_EIA-7343-31_Kemet-D
- removed C34, C35, C37, C38, C39, C41, C42: 10u 35v, Capacitor_SMD:C_0805_2012Metric
- removed C36: 100n 100v, Capacitor_SMD:C_0402_1005Metric
- removed C59, C61: nf, Capacitor_SMD:C_0402_1005Metric
- removed C60: 1.2nF, Capacitor_SMD:C_0402_1005Metric
- removed C8, C9: 27pF, Capacitor_SMD:C_0402_1005Metric
- removed D1: LED Red, LED_SMD:LED_0603_1608Metric
- removed D2: LED Green, LED_SMD:LED_0603_1608Metric
- removed D3: BAT54C-7-F, Package_TO_SOT_SMD:SOT-23
- removed H1, H2, H3, H4: MountingHole, MountingHole:MountingHole_4.3mm_M4
- removed J10, J22: 690-019-298-412, CM4IO:EDAC 690-019-298-412
- removed J11: USB_OTG, CM4IO:USB_Micro-B_EDAC_UCON00686
- removed J13: 690-008-221-904, CM4IO:MOLEX_USB_67298-4090
- removed J14: Conn_02x05_Odd_Even, Connector_PinHeader_2.54mm:PinHeader_2x05_P2.54mm_Vertical
- removed J15, J16, J4, J5: Conn_01x22_Female, CM4IO:Hirose_FH12-22S-0.5SH_1x22-1MP_P0.50mm_Horizontal
- removed J17: Molex 470531000, Connector:FanPinHeader_1x04_P2.54mm_Vertical
- removed J19: Barrel_Jack, CM4IO:BarrelJack_Horizontal
- removed J2: Conn_02x07_Odd_Even, Connector_PinHeader_2.54mm:PinHeader_2x07_P2.54mm_Vertical
- removed J3: Conn_01x03, Connector_PinHeader_2.54mm:PinHeader_1x03_P2.54mm_Vertical
- removed J6, J9: THD-02-R, Connector_PinHeader_2.54mm:PinHeader_2x02_P2.54mm_Vertical
- removed J7: Micro_SD_Card_Det, CM4IO:SDCARD_MOLEX_503398-1892
- removed J8: THD-20-R, Connector_PinHeader_2.54mm:PinHeader_2x20_P2.54mm_Vertical
- removed L5: SRN6045TA-3R3Y, Inductor_SMD:L_Bourns_SRN6045TA
- removed Module1: ComputeModule4, CM4IO:Raspberry-Pi-4-Compute-Module
- removed Q1: DMP3013SFV-7, Package_SON:Diodes_PowerDI3333-8
- removed R1, R10: 1k, Resistor_SMD:R_0402_1005Metric
- removed R11, R28, R6, R7, R8: 2.2K 1%, Resistor_SMD:R_0402_1005Metric
- removed R12, R13, R14, R16, R21: 36K 1%, Resistor_SMD:R_0402_1005Metric
- removed R15, R26, R27, R29: 12K 1%, Resistor_SMD:R_0402_1005Metric
- removed R17, R18: nf, Resistor_SMD:R_0402_1005Metric
- removed R19, R20: 510K 1%, Resistor_SMD:R_0402_1005Metric
- removed R2, R3: 470R, Resistor_SMD:R_0402_1005Metric
- removed R25: 20K 1%, Resistor_SMD:R_0402_1005Metric
- removed R36: 15K 1%, Resistor_SMD:R_0402_1005Metric
- removed R9: 10R, Resistor_SMD:R_0402_1005Metric
- removed TP2, TP3, TP4, TP5, TP6: TestPoint, TestPoint:TestPoint_Pad_2.0x2.0mm
- removed U1, U2, U4: TPD4EUSB30, Package_SON:USON-10_2.5x1.0mm_P0.5mm
- removed U11: EMC2301-1-ACZL-TR, Package_SO:MSOP-8_3x3mm_P0.65mm
- removed U12: RT9742SNGV, Package_TO_SOT_SMD:SOT-23
- removed U13: FSUSB42MUX, Package_SO:MSOP-10_3x3mm_P0.5mm
- removed U14, U5, U9: 74LVC1G07SE-7, Package_TO_SOT_SMD:SOT-353_SC-70-5
- removed U16: AP64501SP-13, Package_SO:SOIC-8-1EP_3.9x4.9mm_P1.27mm_EP2.95x4.9mm_Mask2.71x3.4mm_ThermalVias
- removed U18: RT9742GGJ5, Package_TO_SOT_SMD:SOT-23-5
- removed U3: MagJack-A70-112-331N126, CM4IO:TRJG0926HENL
- removed U6: USB2514B-I/M2, Package_DFN_QFN:QFN-36-1EP_6x6mm_P0.5mm_EP3.7x3.7mm
- removed U7: AP22653W6, Package_TO_SOT_SMD:SOT-23-6
- removed U8: PCF85063AT/AAZ, Package_SO:SOIC-8_3.9x4.9mm_P1.27mm
- removed Y1: 24MHz, Crystal:Crystal_SMD_HC49-SD
- removed Y2: X32K768S301, Crystal:Crystal_SMD_3215-2Pin_3.2x1.5mm
- added M4: MOUNTING, MountingHole:MountingHole_4.3mm_M4, F.Cu at (30.2, 40.8)
- added M5: MOUNTING, MountingHole:MountingHole_4.3mm_M4, F.Cu at (154.2, 40.8)
- added M6: MOUNTING, MountingHole:MountingHole_4.3mm_M4, F.Cu at (30.2, 170.8)
- added M7: MOUNTING, MountingHole:MountingHole_4.3mm_M4, F.Cu at (154.2, 170.8)
- J1: value Conn_01x03 -> SBC; footprint Connector_PinHeader_2.54mm:PinHeader_1x03_P2.54mm_Vertical -> Connector_IDC:IDC-Header_2x13_P2.54mm_Vertical
- moved J1 122.8 mm to (152.9, 94.2)
Connections:
- J1 pad 1: /CM4_GPIO ( Ethernet, GPIO, SDCARD)/GLOBAL_EN -> (no net)
- J1 pad 2: GND -> (no net)
- J1 pad 3: /CM4_GPIO ( Ethernet, GPIO, SDCARD)/RUN_PG -> (no net)

Commit message: complete schematic
Parts:
- removed M4, M5, M7: MOUNTING, MountingHole:MountingHole_4.3mm_M4
- added BT1: Battery_Cell, CM5IO:BatteryHolder_Keystone_3034_1x20mm, F.Cu at (57.5, 100.2)
- added C1: 100n, Capacitor_SMD:C_0402_1005Metric, F.Cu at (169.6, 72.8)
- added C10: 100n, Capacitor_SMD:C_0402_1005Metric, F.Cu at (230.5, 38.3)
- added C11: 10u, Capacitor_SMD:C_0805_2012Metric, F.Cu at (211.9, 67.2)
- added C12: 10u, Capacitor_SMD:C_0805_2012Metric, F.Cu at (216.7, 70.9)
- added C13: 100n, Capacitor_SMD:C_0402_1005Metric, F.Cu at (220.3, 75.3)
- added C14: 4.7nF, Capacitor_SMD:C_0402_1005Metric, F.Cu at (220.3, 77.3)
- added C15: 10u, Capacitor_SMD:C_0805_2012Metric, F.Cu at (216.7, 73.9)
- added C16: 10u, Capacitor_SMD:C_0805_2012Metric, F.Cu at (216.7, 76.9)
- added C17: 10u, Capacitor_SMD:C_0805_2012Metric, F.Cu at (216.7, 79.9)
- added C18: 10u, Capacitor_SMD:C_0805_2012Metric, F.Cu at (216.7, 82.9)
- added C19: 100n, Capacitor_SMD:C_0402_1005Metric, F.Cu at (220.3, 79.3)
- added C2: 100n, Capacitor_SMD:C_0402_1005Metric, F.Cu at (169.6, 74.7)
- added C20: 10uF, Capacitor_SMD:C_1210_3225Metric_Pad1.33x2.70mm_HandSolder, F.Cu at (133.7, 68.3)
- added C3: 10u, Capacitor_SMD:C_0805_2012Metric, F.Cu at (238.5, 73.7)
- added C4: 100uF, Capacitor_Tantalum_SMD:CP_EIA-7343-31_Kemet-D, F.Cu at (234.0, 69.3)
- added C5: 10u, Capacitor_SMD:C_0805_2012Metric, F.Cu at (238.5, 76.7)
- added C6: 10u, Capacitor_SMD:C_0805_2012Metric, F.Cu at (238.5, 79.8)
- added C7: 100n, Capacitor_SMD:C_0402_1005Metric, F.Cu at (242.1, 81.2)
- added C8: 100n, Capacitor_SMD:C_0402_1005Metric, F.Cu at (242.1, 83.1)
- added C9: 10u, Capacitor_SMD:C_0805_2012Metric, F.Cu at (226.8, 38.8)
- added D1: LED Green, LED_SMD:LED_0603_1608Metric, F.Cu at (230.0, 41.9)
- added D2: LED Red, LED_SMD:LED_0603_1608Metric, F.Cu at (230.0, 44.5)
- added D3: LED Green, LED_SMD:LED_0603_1608Metric, F.Cu at (223.8, 72.1)
- added D4: D_Schottky, Diode_SMD:D_SMA_Handsoldering, F.Cu at (131.0, 74.9)
- added F1: MCCQ-122, footprints:MCCQ-122, F.Cu at (98.8, 62.8)
- added F2: MCCQ-122, footprints:MCCQ-122, F.Cu at (79.8, 62.8)
- added F3: MCCQ-122, footprints:MCCQ-122, F.Cu at (60.9, 62.8)
- added H1: ~, MountingHole:MountingHole_4.3mm_M4, F.Cu at (30.2, 40.8)
- added H2: ~, MountingHole:MountingHole_4.3mm_M4, F.Cu at (154.2, 40.8)
- added H3: ~, MountingHole:MountingHole_4.3mm_M4, F.Cu at (30.2, 170.8)
- added H4: ~, MountingHole:MountingHole_4.3mm_M4, F.Cu at (154.2, 170.8)
- added J10: JST_SHBM04B-SRSS-TB, Connector_JST:JST_SH_BM04B-SRSS-TB_1x04-1MP_P1.00mm_Vertical, F.Cu at (60.2, 122.8)
- added J11: THD-20-R, Connector_PinHeader_2.54mm:PinHeader_2x20_P2.54mm_Vertical, F.Cu at (38.9, 95.4)
- added J12: THD-02-R, Connector_PinHeader_2.54mm:PinHeader_2x02_P2.54mm_Vertical, F.Cu at (52.9, 75.4)
- added J13: Micro_SD_Card_Det, CM5IO:SDCARD_MOLEX_503398-1892, F.Cu at (152.1, 66.5)
- added J14: Bus_M.2_Socket_M, CM5IO:M.2 M Key socket, F.Cu at (126.8, 153.0)
- added J16: THD-20-R, Connector_IDC:IDC-Header_2x13_P2.54mm_Vertical, B.Cu at (31.5, 94.2)
- added J17: HB9500-9.5-8P, footprints:HB9500-9.5-8P, F.Cu at (45.8, 53.8)
- added J2: Conn_01x22_Female, CM5IO:Hirose_FH12-22S-0.5SH_1x22-1MP_P0.50mm_Horizontal, F.Cu at (154.8, 112.8)
- added J3: Conn_01x22_Female, CM5IO:Hirose_FH12-22S-0.5SH_1x22-1MP_P0.50mm_Horizontal, F.Cu at (46.5, 171.1)
- added J4: THD-02-R, Connector_PinHeader_2.54mm:PinHeader_2x02_P2.54mm_Vertical, F.Cu at (231.4, 74.5)
- added J5: USB3_A, CM5IO:MTCONN_UBAF30-D2011, F.Cu at (149.5, 132.7)
- added J6: 690-019-298-412, CM5IO:EDAC 690-019-298-412, F.Cu at (149.0, 153.1)
- added J7: 690-019-298-412, CM5IO:EDAC 690-019-298-412, F.Cu at (35.7, 156.4)
- added J8: Conn_02x07_Odd_Even, Connector_PinHeader_2.54mm:PinHeader_2x07_P2.54mm_Vertical, F.Cu at (124.4, 97.1)
- added J9: Conn_01x03, Connector_PinHeader_2.54mm:PinHeader_1x03_P2.54mm_Vertical, F.Cu at (135.7, 103.8)
- added L1: 2.2uH, CM5IO:L_Bourns_SRP5030CC, F.Cu at (135.6, 133.2)
- added L2: 8.2uH, footprints:SMD_inductor_07A7, F.Cu at (127.4, 81.0)
- added Module1: ComputeModule5-CM5, CM5IO:Raspberry-Pi-5-Compute-Module, B.Cu at (66.4, 170.0)
- added R1: 2.2K 1%, Resistor_SMD:R_0402_1005Metric, F.Cu at (38.8, 56.4)
- added R10: 470R, Resistor_SMD:R_0402_1005Metric, F.Cu at (230.1, 10.5)
- added R11: 470R, Resistor_SMD:R_0402_1005Metric, F.Cu at (230.1, 12.5)
- added R12: 100K 1%, Resistor_SMD:R_0402_1005Metric, F.Cu at (220.3, 67.4)
- added R13: 10K 1%, Resistor_SMD:R_0402_1005Metric, F.Cu at (220.3, 69.4)
- added R14: 2.2K 1%, Resistor_SMD:R_0402_1005Metric, F.Cu at (220.3, 71.3)
- added R15: 1k, Resistor_SMD:R_0402_1005Metric, F.Cu at (220.3, 73.3)
- added R2: 15K 1%, Resistor_SMD:R_0402_1005Metric, F.Cu at (242.1, 73.2)
- added R3: 2.2K 1%, Resistor_SMD:R_0402_1005Metric, F.Cu at (242.1, 75.2)
- added R4: 2.2K 1%, Resistor_SMD:R_0402_1005Metric, F.Cu at (242.1, 77.2)
- added R5: 2.2K 1%, Resistor_SMD:R_0402_1005Metric, F.Cu at (242.1, 79.2)
- added R6: 1k, Resistor_SMD:R_0402_1005Metric, F.Cu at (230.1, 6.54)
- added R7: 0R, Resistor_SMD:R_0805_2012Metric_Pad1.20x1.40mm_HandSolder, F.Cu at (219.8, 42.0)
- added R8: nf, Resistor_SMD:R_0805_2012Metric_Pad1.20x1.40mm_HandSolder, F.Cu at (219.8, 45.0)
- added R9: 1k, Resistor_SMD:R_0402_1005Metric, F.Cu at (230.1, 8.54)
- added SW1: Right angle Tact button, Button_Switch_THT:SW_Tactile_SPST_Angled_PTS645Vx58-2LFS, F.Cu at (129.9, 173.4)
- added TP1: TestPoint, TestPoint:TestPoint_Pad_2.0x2.0mm, F.Cu at (246.3, 36.1)
- added TP2: TestPoint, TestPoint:TestPoint_Pad_2.0x2.0mm, F.Cu at (226.6, 11.6)
- added TP3: TestPoint, TestPoint:TestPoint_Pad_2.0x2.0mm, F.Cu at (223.8, 76.4)
- added U1: AP22653W6, Package_TO_SOT_SMD:SOT-23-6, F.Cu at (142.9, 117.2)
- added U10: LV14360, footprints:LV14360, F.Cu at (123.2, 66.4)
- added U2: RT9742SNGV, Package_TO_SOT_SMD:TSOT-23_HandSoldering, F.Cu at (232.5, 81.9)
- added U3: 74LVC1G07SE-7, Package_TO_SOT_SMD:SOT-353_SC-70-5, F.Cu at (226.7, 35.4)
- added U4: TPD4EUSB30, Package_SON:USON-10_2.5x1.0mm_P0.5mm, F.Cu at (223.6, 42.8)
- added U5: TPD4EUSB30, Package_SON:USON-10_2.5x1.0mm_P0.5mm, F.Cu at (226.5, 42.8)
- added U6: RT9742GGJ5, Package_TO_SOT_SMD:SOT-23-5, F.Cu at (228.8, 29.5)
- added U7: MagJack-A70-112-331N126, CM5IO:TRJG0926HENL, F.Cu at (36.3, 74.1)
- added U8: AP3441SHE-7B, Package_DFN_QFN:DFN-8-1EP_2x2mm_P0.5mm_EP1.05x1.75mm, F.Cu at (127.8, 127.8)
- added U9: ASEK-32.768KHZ-L-R-T, Crystal:Crystal_SMD_3225-4Pin_3.2x2.5mm, F.Cu at (224.4, 68.6)
- J1: value SBC -> USB_C_Receptacle_USB2.0; footprint Connector_IDC:IDC-Header_2x13_P2.54mm_Vertical -> Connector_USB:USB_C_Receptacle_GCT_USB4105-xx-A_16P_TopMnt_Horizontal
- M6: value MOUNTING -> Fan; footprint MountingHole:MountingHole_4.3mm_M4 -> footprints:fan_40mm_M3
- moved J1 129.1 mm to (29.0, 58.2), turned to -90 degrees
- moved M6 91.6 mm to (94.4, 105.3)
Routing:
- net /CM5_HighSpeed/PCIE_nWAKE: track 0.00 -> 1.03 mm

Commit message: stalled routing
Parts:
- removed the C7 at (242.1, 81.2)
- removed the C8 at (242.1, 83.1)
- removed the J12 at (52.9, 75.4)
- removed the R7 at (219.8, 42.0)
- removed the R8 at (219.8, 45.0)
- removed the U2 at (232.5, 81.9)
- added AE1: SR4W035, footprints:SR4W035, F.Cu at (149.5, 56.5)
- added C21: 10uF, Capacitor_SMD:C_1210_3225Metric_Pad1.33x2.70mm_HandSolder, F.Cu at (61.8, 92.6)
- added C22: 0.1uF, Capacitor_SMD:C_0805_2012Metric_Pad1.18x1.45mm_HandSolder, F.Cu at (61.5, 95.9)
- added C23: 100n, Capacitor_SMD:C_0805_2012Metric_Pad1.18x1.45mm_HandSolder, F.Cu at (65.4, 101.0)
- added C24: 10uF, Capacitor_SMD:C_1210_3225Metric_Pad1.33x2.70mm_HandSolder, F.Cu at (53.4, 107.9)
- added C25: 10uF, Capacitor_SMD:C_1210_3225Metric_Pad1.33x2.70mm_HandSolder, F.Cu at (53.4, 111.9)
- added C26: 10uF, Capacitor_SMD:C_1210_3225Metric_Pad1.33x2.70mm_HandSolder, F.Cu at (53.4, 115.3)
- added C27: 10000pF, Capacitor_SMD:C_0805_2012Metric_Pad1.18x1.45mm_HandSolder, F.Cu at (53.3, 92.9)
- added C28: 47pF, Capacitor_SMD:C_0805_2012Metric_Pad1.18x1.45mm_HandSolder, F.Cu at (69.1, 120.6)
- added C29: 4.7nF, Capacitor_SMD:C_0805_2012Metric_Pad1.18x1.45mm_HandSolder, F.Cu at (65.4, 123.1)
- added C30: C, Capacitor_SMD:C_0805_2012Metric, F.Cu at (145.9, 55.2)
- added C31: 10uF, Capacitor_SMD:C_1210_3225Metric_Pad1.33x2.70mm_HandSolder, F.Cu at (124.7, 65.5)
- added C32: 10uF, Capacitor_SMD:C_1210_3225Metric_Pad1.33x2.70mm_HandSolder, F.Cu at (124.7, 61.8)
- added C33: 0.1uF, Capacitor_SMD:C_0805_2012Metric_Pad1.18x1.45mm_HandSolder, F.Cu at (124.9, 68.7)
- added C34: 100n, Capacitor_SMD:C_0805_2012Metric_Pad1.18x1.45mm_HandSolder, F.Cu at (130.7, 68.3)
- added C35: 10uF, Capacitor_SMD:C_1210_3225Metric_Pad1.33x2.70mm_HandSolder, F.Cu at (104.7, 81.4)
- added C36: 10uF, Capacitor_SMD:C_1210_3225Metric_Pad1.33x2.70mm_HandSolder, F.Cu at (109.3, 81.4)
- added C37: 10uF, Capacitor_SMD:C_1210_3225Metric_Pad1.33x2.70mm_HandSolder, F.Cu at (100.1, 81.4)
- added C38: 10000pF, Capacitor_SMD:C_0805_2012Metric_Pad1.18x1.45mm_HandSolder, F.Cu at (134.8, 73.6)
- added C39: 47pF, Capacitor_SMD:C_0805_2012Metric_Pad1.18x1.45mm_HandSolder, F.Cu at (136.9, 73.5)
- added C40: 4.7nF, Capacitor_SMD:C_0805_2012Metric_Pad1.18x1.45mm_HandSolder, F.Cu at (139.1, 71.5)
- added C5: 100n, Capacitor_SMD:C_0805_2012Metric_Pad1.18x1.45mm_HandSolder, F.Cu at (31.2, 137.9)
- added C6: 100n, Capacitor_SMD:C_0805_2012Metric_Pad1.18x1.45mm_HandSolder, F.Cu at (31.0, 144.2)
- added D5: D_Schottky, Diode_SMD:D_SMA_Handsoldering, F.Cu at (127.2, 79.3)
- added F4: MCCQ-122, footprints:MCCQ-122, F.Cu at (57.7, 65.3)
- added J16: Screw_Terminal_01x10, footprints:HB9500-9.5-10p, F.Cu at (42.3, 54.2)
- added JP1: SolderJumper_3_Bridged12, Jumper:SolderJumper-3_P1.3mm_Bridged12_RoundedPad1.0x1.5mm, F.Cu at (99.9, 143.4)
- added JP2: SolderJumper_3_Open, footprints:resistor_jumper_3_way_0805, F.Cu at (104.8, 66.4)
- added JP3: SolderJumper_3_Open, footprints:resistor_jumper_3_way_0805, F.Cu at (86.4, 66.4)
- added JP4: SolderJumper_3_Open, footprints:resistor_jumper_3_way_0805, F.Cu at (66.1, 66.4)
- added JP5: SolderJumper_3_Open, footprints:resistor_jumper_3_way_0805, F.Cu at (47.4, 66.4)
- added L3: 2.2nH, Inductor_SMD:L_0805_2012Metric_Pad1.05x1.20mm_HandSolder, F.Cu at (150.0, 51.2)
- added L4: 2.2nH, Inductor_SMD:L_0805_2012Metric_Pad1.05x1.20mm_HandSolder, F.Cu at (146.0, 52.8)
- added L5: 8.2uH, footprints:SMD_inductor_07A7, F.Cu at (121.4, 77.6)
- added R14: R, Resistor_SMD:R_0805_2012Metric_Pad1.20x1.40mm_HandSolder, F.Cu at (49.0, 88.0)
- added R15: R, Resistor_SMD:R_0805_2012Metric_Pad1.20x1.40mm_HandSolder, F.Cu at (53.0, 88.0)
- added R16: 100k, Resistor_SMD:R_0805_2012Metric_Pad1.20x1.40mm_HandSolder, F.Cu at (55.0, 104.3)
- added R17: 240k, Resistor_SMD:R_0805_2012Metric_Pad1.20x1.40mm_HandSolder, F.Cu at (53.2, 96.5)
- added R18: 19.1k, Resistor_SMD:R_0805_2012Metric_Pad1.20x1.40mm_HandSolder, F.Cu at (54.9, 100.3)
- added R19: 3.24k, Resistor_SMD:R_0805_2012Metric_Pad1.20x1.40mm_HandSolder, F.Cu at (65.5, 118.5)
- added R20: R, Resistor_SMD:R_0805_2012Metric_Pad1.20x1.40mm_HandSolder, F.Cu at (140.7, 62.6)
- added R21: R, Resistor_SMD:R_0805_2012Metric_Pad1.20x1.40mm_HandSolder, F.Cu at (121.5, 72.9)
- added R22: R, Resistor_SMD:R_0805_2012Metric_Pad1.20x1.40mm_HandSolder, F.Cu at (125.4, 73.8)
- added R23: 100k, Resistor_SMD:R_0805_2012Metric_Pad1.20x1.40mm_HandSolder, F.Cu at (117.8, 83.5)
- added R24: 240k, Resistor_SMD:R_0805_2012Metric_Pad1.20x1.40mm_HandSolder, F.Cu at (123.9, 76.0)
- added R25: 3.24k, Resistor_SMD:R_0805_2012Metric_Pad1.20x1.40mm_HandSolder, F.Cu at (117.8, 87.9)
- added R26: 3.24k, Resistor_SMD:R_0805_2012Metric_Pad1.20x1.40mm_HandSolder, F.Cu at (139.0, 75.4)
- added U11: TPP60508, footprints:DFN-10_EP_4x4_Pitch0.8mm, F.Cu at (130.5, 72.1)
- added U6: RT9742SNGV, Package_TO_SOT_SMD:TSOT-23_HandSoldering, F.Cu at (31.2, 141.1)
- C1, C2: footprint Capacitor_SMD:C_0402_1005Metric -> Capacitor_SMD:C_0805_2012Metric_Pad1.18x1.45mm_HandSolder
- C10: renamed from C6; footprint Capacitor_SMD:C_0805_2012Metric -> Capacitor_SMD:C_0805_2012Metric_Pad1.18x1.45mm_HandSolder
- C11: renamed from C19; footprint Capacitor_SMD:C_0402_1005Metric -> Capacitor_SMD:C_0805_2012Metric_Pad1.18x1.45mm_HandSolder
- C12: renamed from C11; footprint Capacitor_SMD:C_0805_2012Metric -> Capacitor_SMD:C_0805_2012Metric_Pad1.18x1.45mm_HandSolder
- C13: renamed from C12; footprint Capacitor_SMD:C_0805_2012Metric -> Capacitor_SMD:C_0805_2012Metric_Pad1.18x1.45mm_HandSolder
- C14: renamed from C13; footprint Capacitor_SMD:C_0402_1005Metric -> Capacitor_SMD:C_0805_2012Metric_Pad1.18x1.45mm_HandSolder
- C15: renamed from C14; footprint Capacitor_SMD:C_0402_1005Metric -> Capacitor_SMD:C_0805_2012Metric_Pad1.18x1.45mm_HandSolder
- C16: renamed from C15; footprint Capacitor_SMD:C_0805_2012Metric -> Capacitor_SMD:C_0805_2012Metric_Pad1.18x1.45mm_HandSolder
- C17: renamed from C16; footprint Capacitor_SMD:C_0805_2012Metric -> Capacitor_SMD:C_0805_2012Metric_Pad1.18x1.45mm_HandSolder
- C18: renamed from C17; footprint Capacitor_SMD:C_0805_2012Metric -> Capacitor_SMD:C_0805_2012Metric_Pad1.18x1.45mm_HandSolder
- C19: renamed from C18; footprint Capacitor_SMD:C_0805_2012Metric -> Capacitor_SMD:C_0805_2012Metric_Pad1.18x1.45mm_HandSolder
- C3: renamed from C10; footprint Capacitor_SMD:C_0402_1005Metric -> Capacitor_SMD:C_0805_2012Metric_Pad1.18x1.45mm_HandSolder
- C4: renamed from C9; footprint Capacitor_SMD:C_0805_2012Metric -> Capacitor_SMD:C_0805_2012Metric_Pad1.18x1.45mm_HandSolder
- C7: renamed from C3; footprint Capacitor_SMD:C_0805_2012Metric -> Capacitor_SMD:C_0805_2012Metric_Pad1.18x1.45mm_HandSolder
- C9: renamed from C5; footprint Capacitor_SMD:C_0805_2012Metric -> Capacitor_SMD:C_0805_2012Metric_Pad1.18x1.45mm_HandSolder
- J17: value HB9500-9.5-8P -> Conn_Coaxial; footprint footprints:HB9500-9.5-8P -> Connector_Coaxial:U.FL_Hirose_U.FL-R-SMT-1_Vertical
- J7: renamed from J10; value JST_SHBM04B-SRSS-TB -> ~; footprint Connector_JST:JST_SH_BM04B-SRSS-TB_1x04-1MP_P1.00mm_Vertical -> Connector:FanPinHeader_1x04_P2.54mm_Vertical
- R1, R12: footprint Resistor_SMD:R_0402_1005Metric -> Resistor_SMD:R_0805_2012Metric_Pad1.20x1.40mm_HandSolder
- R10: renamed from R15; footprint Resistor_SMD:R_0402_1005Metric -> Resistor_SMD:R_0805_2012Metric_Pad1.20x1.40mm_HandSolder
- R11: renamed from R13; footprint Resistor_SMD:R_0402_1005Metric -> Resistor_SMD:R_0805_2012Metric_Pad1.20x1.40mm_HandSolder
- R13: renamed from R14; footprint Resistor_SMD:R_0402_1005Metric -> Resistor_SMD:R_0805_2012Metric_Pad1.20x1.40mm_HandSolder
- R2: renamed from R6; footprint Resistor_SMD:R_0402_1005Metric -> Resistor_SMD:R_0805_2012Metric_Pad1.20x1.40mm_HandSolder
- R3: renamed from R10; footprint Resistor_SMD:R_0402_1005Metric -> Resistor_SMD:R_0805_2012Metric_Pad1.20x1.40mm_HandSolder
- R4: renamed from R11; footprint Resistor_SMD:R_0402_1005Metric -> Resistor_SMD:R_0805_2012Metric_Pad1.20x1.40mm_HandSolder
- R5: renamed from R9; footprint Resistor_SMD:R_0402_1005Metric -> Resistor_SMD:R_0805_2012Metric_Pad1.20x1.40mm_HandSolder
- R6: renamed from R4; footprint Resistor_SMD:R_0402_1005Metric -> Resistor_SMD:R_0805_2012Metric_Pad1.20x1.40mm_HandSolder
- R7: renamed from R5; footprint Resistor_SMD:R_0402_1005Metric -> Resistor_SMD:R_0805_2012Metric_Pad1.20x1.40mm_HandSolder
- R8: renamed from R3; footprint Resistor_SMD:R_0402_1005Metric -> Resistor_SMD:R_0805_2012Metric_Pad1.20x1.40mm_HandSolder
- R9: renamed from R2; footprint Resistor_SMD:R_0402_1005Metric -> Resistor_SMD:R_0805_2012Metric_Pad1.20x1.40mm_HandSolder
- U10: value LV14360 -> TPP60508; footprint footprints:LV14360 -> footprints:DFN-10_EP_4x4_Pitch0.8mm
- moved R6 219.2 mm to (41.2, 164.9), turned to -90 degrees
- moved R7 216.6 mm to (43.2, 164.9), turned to -90 degrees
- moved R3 214.0 mm to (29.2, 84.3), turned to -90 degrees
- moved R4 210.2 mm to (32.5, 84.5), turned to -90 degrees
- moved J12 200.6 mm to (44.0, 146.2), turned to -90 degrees
- moved R2 185.4 mm to (142.2, 169.8)
- moved U1 185.0 mm to (43.4, 85.1), turned to -90 degrees
- moved U2 183.8 mm to (43.9, 63.8), turned to 90 degrees
- moved TP1 166.9 mm to (141.4, 165.9)
- moved D1 157.6 mm to (138.0, 169.8), turned to 180 degrees
- moved C1 135.4 mm to (36.0, 50.8), turned to 180 degrees
- moved C2 131.0 mm to (39.4, 61.0)
- moved U8 125.3 mm to (137.2, 158.4)
- moved D3 119.9 mm to (136.0, 153.7), turned to 90 degrees
- moved C11 117.9 mm to (137.0, 162.7)
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- renumbered C4 to C8, J6 to J10, J5 to J11, J4 to J12, J3 to J13, J7 to J14, J14 to J15, J11 to J2, J16 to J4, J13 to J5, J9 to J6, J2 to J9, U4 to U1, U5 to U2, U7 to U3, U3 to U4, U6 to U5, U1 to U7, U9 to U8, U8 to U9
Connections:
- C20 pad 1: Net-(U10-PGOOD) -> /misc/Vin
- F1 pad 1: Net-(J17-Pin_6) -> Net-(J16-Pin_8)
- F1 pad 2: /misc/Vin -> Net-(JP2-C)
- F2 pad 1: Net-(J17-Pin_4) -> Net-(J16-Pin_6)
- F2 pad 2: /misc/Vin -> Net-(JP3-C)
- F3 pad 1: Net-(J17-Pin_2) -> Net-(J16-Pin_4)
- F3 pad 2: /misc/Vin -> Net-(JP4-C)
- J17 pad 1: GND -> Net-(J17-In)
- J17 pad 2: Net-(J17-Pin_2) -> Net-(J17-Ext)
- U10 pad 3: /misc/Vin -> Net-(U10-EN)
- U10 pad 6: Net-(U10-PGOOD) -> Net-(U10-FB)
- U10 pad 7: GND -> Net-(U10-COMP)
- U10 pad 8: Net-(D4-K) -> GND
- U10 pad 9: GND -> Net-(D4-K)
Routing:
- net GND: track 0.00 -> 265.5 mm, vias 0 -> 22
- net /misc/Vin: track 0.00 -> 159.9 mm
- net /CM5_HighSpeed/DPHY0_D2_N: track 0.00 -> 95.8 mm, vias 0 -> 3
- net /CM5_HighSpeed/DPHY0_D2_P: track 0.00 -> 95.8 mm, vias 0 -> 3
- net /CM5_GPIO ( Ethernet, GPIO, SDCARD)/SD_DAT2: track 0.00 -> 94.0 mm, vias 0 -> 1
- net /CM5_HighSpeed/DPHY0_D3_N: track 0.00 -> 93.2 mm, vias 0 -> 3
- net /CM5_HighSpeed/DPHY0_D3_P: track 0.00 -> 93.2 mm, vias 0 -> 3
- net /CM5_HighSpeed/DPHY0_D0_N: track 0.00 -> 92.6 mm, vias 0 -> 3
- net /CM5_HighSpeed/DPHY0_D0_P: track 0.00 -> 92.5 mm, vias 0 -> 3
- net /CM5_HighSpeed/DPHY0_D1_N: track 0.00 -> 90.4 mm, vias 0 -> 3
- net /CM5_HighSpeed/DPHY0_D1_P: track 0.00 -> 90.4 mm, vias 0 -> 3
- net /misc/Vreg2: track 0.00 -> 90.0 mm
- net /CM5_HighSpeed/DPHY0_C_N: track 0.00 -> 88.3 mm, vias 0 -> 3
- net /CM5_HighSpeed/DPHY0_C_P: track 0.00 -> 88.3 mm, vias 0 -> 3
- net /CM5_HighSpeed/USB3-0-RX_N: track 0.00 -> 86.2 mm, vias 0 -> 2
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- added copper zone on In1.Cu, net GND
- added copper zone on In2.Cu, net GND
Other:
- copper layers 2 -> 4
- board text added: "WayWayWay"

Commit message: pre-revise 5v route
Parts:
- removed AE1: SR4W035, footprints:SR4W035
- removed C30: C, Capacitor_SMD:C_0805_2012Metric
- removed J17: Conn_Coaxial, Connector_Coaxial:U.FL_Hirose_U.FL-R-SMT-1_Vertical
- removed L3, L4: 2.2nH, Inductor_SMD:L_0805_2012Metric_Pad1.05x1.20mm_HandSolder
- removed R20: R, Resistor_SMD:R_0805_2012Metric_Pad1.20x1.40mm_HandSolder
- BT1, J15, JP1, JP2, JP3, JP4, JP5: moved to B.Cu
- J14: footprint CM5IO:EDAC 690-019-298-412 -> Connector_Video:HDMI_Micro-D_Molex_46765-1x01
- Module1: moved to F.Cu
- moved C4 167.0 mm to (55.2, 172.3), turned to -90 degrees
- moved C3 157.9 mm to (49.6, 71.0)
- moved R5 152.3 mm to (82.0, 172.3), turned to -90 degrees
- moved U4 152.3 mm to (73.9, 171.8)
- moved J5 146.6 mm to (46.9, 168.6), turned to 180 degrees
- moved TP2 145.5 mm to (77.5, 173.6), turned to -90 degrees
- moved D2 144.0 mm to (77.3, 171.1), turned to 180 degrees
- moved BT1 129.2 mm to (71.4, 192.7), turned to 180 degrees
- moved J14 121.7 mm to (156.1, 138.8), turned to 90 degrees
- moved U5 118.9 mm to (56.3, 167.8), turned to 90 degrees
- moved J1 118.8 mm to (64.2, 171.6), turned to 0 degrees
- moved C1 117.7 mm to (60.8, 165.8)
- moved R1 117.1 mm to (71.0, 169.0), turned to 90 degrees
- moved R8 115.1 mm to (108.0, 171.4)
- moved C6 109.9 mm to (139.7, 159.8), turned to 90 degrees
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Routing:
- net /+5v: track 53.5 -> 328.3 mm, vias 0 -> 16
- net /+3.3v: track 26.4 -> 268.5 mm, vias 0 -> 5
- net /CM5_GPIO ( Ethernet, GPIO, SDCARD)/ID_SC: track 0.00 -> 201.2 mm, vias 0 -> 4
- net /CM5_GPIO ( Ethernet, GPIO, SDCARD)/ID_SD: track 0.00 -> 198.6 mm, vias 0 -> 4
- net /CM5_GPIO ( Ethernet, GPIO, SDCARD)/GPIO21: track 0.00 -> 146.9 mm
- net /CM5_GPIO ( Ethernet, GPIO, SDCARD)/GPIO26: track 0.00 -> 144.4 mm, vias 0 -> 2
- net /CM5_GPIO ( Ethernet, GPIO, SDCARD)/GPIO20: track 0.00 -> 143.6 mm
- net /CM5_GPIO ( Ethernet, GPIO, SDCARD)/GPIO19: track 0.00 -> 143.1 mm, vias 0 -> 2
- net /CM5_GPIO ( Ethernet, GPIO, SDCARD)/GPIO16: track 0.00 -> 140.5 mm
- net /CM5_GPIO ( Ethernet, GPIO, SDCARD)/GPIO13: track 0.00 -> 138.5 mm, vias 0 -> 2
- net /CM5_GPIO ( Ethernet, GPIO, SDCARD)/GPIO12: track 0.00 -> 135.8 mm
- net /CM5_GPIO ( Ethernet, GPIO, SDCARD)/GPIO6: track 0.00 -> 135.4 mm, vias 0 -> 2
- net /CM5_GPIO ( Ethernet, GPIO, SDCARD)/GPIO5: track 0.00 -> 130.5 mm, vias 0 -> 2
- net /CM5_GPIO ( Ethernet, GPIO, SDCARD)/GPIO7: track 13.4 -> 137.1 mm
- net /CM5_GPIO ( Ethernet, GPIO, SDCARD)/GPIO11: track 7.40 -> 128.7 mm, vias 0 -> 2
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- added copper zone on F.Cu, net /misc/Vin
- added copper zone on In2.Cu, net /misc/Vreg2
Other:
- board text added: "Duet Pi Rev New"
- board text added: "JMP: disable eMMC Boot"
- board text added: "JMP: disable writing to EEPROM"
- board text added: "PMIC_Enable"
- board text added: "PWR_Button"
- board text added: "SYNC_Out"
- board text added: "USB_OTG"

Commit message: finding a home for the battery
Parts:
- moved J6 101.0 mm to (139.8, 168.0)
- moved BT1 16.8 mm to (88.0, 189.9)
- moved J7 0.85 mm to (66.4, 88.4), turned to -90 degrees
- moved C6 0.64 mm to (140.4, 159.9)
- moved U6 0.64 mm to (136.9, 159.9)
- moved C5 0.64 mm to (134.0, 159.7)
Routing:
- net /+5v: track 328.3 -> 526.8 mm, vias 16 -> 17
- net /CM5_GPIO ( Ethernet, GPIO, SDCARD)/PWR_BUT: track 27.1 -> 118.5 mm, vias 0 -> 2
- net GND: track 312.3 -> 398.2 mm, vias 137 -> 144
- net /CM5_GPIO ( Ethernet, GPIO, SDCARD)/BT_nDis: track 0.00 -> 80.4 mm, vias 0 -> 2
- net /CM5_GPIO ( Ethernet, GPIO, SDCARD)/nRPIBOOT: track 53.7 -> 133.4 mm, vias 0 -> 2
- net /CM5_GPIO ( Ethernet, GPIO, SDCARD)/WL_nDis: track 0.00 -> 76.6 mm, vias 0 -> 2
- net /CM5_GPIO ( Ethernet, GPIO, SDCARD)/PMIC_ENABLE: track 41.5 -> 116.7 mm, vias 1 -> 2
- net /CM5_GPIO ( Ethernet, GPIO, SDCARD)/PWM: track 0.00 -> 59.2 mm, vias 0 -> 1
- net /CM5_GPIO ( Ethernet, GPIO, SDCARD)/TACHO: track 0.00 -> 56.8 mm
- net (no net): track 0.00 -> 24.7 mm
- net Net-(R5-Pad2): track 0.00 -> 9.27 mm
- net Net-(J15-DAS/~{DSS}/~{LED1}): track 18.1 -> 10.2 mm
- net Net-(D2-K): track 0.00 -> 6.71 mm
- net /CM5_HighSpeed/PCIE_nCLKREQ: track 57.1 -> 63.5 mm, vias 1 -> 3
- net /CM5_HighSpeed/PCIE_nWAKE: track 58.4 -> 64.4 mm
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Other:
- board text added: "Duet3 Pi v0.1"
- board text removed: "Duet Pi Rev New"

Commit message: everything routed, 4 errors
Parts:
- moved BT1 49.1 mm to (57.8, 151.2), turned to 90 degrees
Routing:
- net /CM5_HighSpeed/PCIE_PWR_EN: track 6.63 -> 142.4 mm, vias 0 -> 4
- net /CM5_GPIO ( Ethernet, GPIO, SDCARD)/VBAT: track 0.00 -> 77.4 mm, vias 0 -> 1
- net /+5v: track 526.8 -> 501.0 mm, vias 17 -> 16
- net (no net): track 24.7 -> 0.00 mm
- net Net-(Module1A-LED_nACT): track 26.1 -> 40.7 mm
- net /+3.3v: track 272.7 -> 281.2 mm
- net /PCIe-M2/M2_3v3: track 79.8 -> 76.1 mm
- net /CM5_GPIO ( Ethernet, GPIO, SDCARD)/CAM_GPIO0: track 26.2 -> 27.2 mm
- net GND: track 398.2 -> 399.0 mm, vias 144 -> 146
- net /CM5_GPIO ( Ethernet, GPIO, SDCARD)/SD_CMD: track 66.5 -> 65.9 mm
- net /CM5_GPIO ( Ethernet, GPIO, SDCARD)/nPWR_LED: track 35.7 -> 36.3 mm

Commit message: differential pair matching
Routing:
- net /CM5_HighSpeed/PCIE_RX_P: track 93.1 -> 105.4 mm
- net /CM5_HighSpeed/PCIE_RX_N: track 95.7 -> 107.9 mm
- net /CM5_HighSpeed/DPHY1_C_N: track 24.3 -> 34.1 mm
- net /CM5_HighSpeed/DPHY1_C_P: track 23.8 -> 33.4 mm
- net /CM5_HighSpeed/DPHY0_D1_P: track 51.4 -> 59.3 mm
- net /CM5_HighSpeed/DPHY0_D1_N: track 51.4 -> 59.3 mm
- net /CM5_HighSpeed/DPHY1_D1_P: track 25.8 -> 33.0 mm
- net /CM5_HighSpeed/DPHY1_D1_N: track 26.3 -> 33.0 mm
- net /CM5_HighSpeed/PCIE_CLK_P: track 103.9 -> 109.1 mm
- net /CM5_HighSpeed/PCIE_CLK_N: track 102.7 -> 107.9 mm
- net /CM5_HighSpeed/DPHY0_C_N: track 56.9 -> 59.1 mm
- net /CM5_HighSpeed/DPHY0_C_P: track 56.9 -> 59.1 mm
- net /CM5_HighSpeed/DPHY1_D2_P: track 33.1 -> 34.6 mm
- net /CM5_HighSpeed/DPHY0_D2_P: track 58.8 -> 59.9 mm
- net /CM5_HighSpeed/DPHY0_D2_N: track 58.7 -> 59.9 mm
