File: duet_pi.kicad_pcb (KiCad board)
At the start: 4 copper layers, 134 x 140 mm, 118 parts, among them J1 USB_C_Receptacle_USB2.0, J10 690-019-298-412, J11 USB3_A, J12 THD-02-R, J13 Conn_01x22_Female, J14 690-019-298-412, J15 Bus_M.2_Socket_M, J16 Screw_Terminal_01x10, J2 THD-20-R, J4 THD-20-R, J5 Micro_SD_Card_Det, J6 Conn_01x03, J8 Conn_02x07_Odd_Even, J9 Conn_01x22_Female, M6 Fan, SW1 Right angle Tact button, U1 TPD4EUSB30, U10 TPP60508, U11 TPP60508, U2 TPD4EUSB30, U3 MagJack-A70-112-331N126, U4 74LVC1G07SE-7, U5 RT9742GGJ5, U6 RT9742SNGV, U7 AP22653W6, U8 ASEK-32.768KHZ-L-R-T, U9 AP3441SHE-7B

Commit message: nearing final routing
Parts:
- added JP6: SolderJumper_3_Open, Jumper:SolderJumper-3_P1.3mm_Open_RoundedPad1.0x1.5mm, B.Cu at (122.5, 71.5)
- added R27: 10.5k, Resistor_SMD:R_0805_2012Metric_Pad1.20x1.40mm_HandSolder, F.Cu at (120.7, 67.8)
- R16, R23: value 100k -> 147k
- R18: value 19.1k -> 28k
- R25: value 3.24k -> 5.05k
- moved R25 4.59 mm to (123.4, 67.8), turned to -90 degrees
Connections:
- R23 pad 1: Net-(U11-FB) -> Net-(JP6-C)
- R25 pad 2: Net-(U11-FB) -> /misc/R_fb_24
- U11 pad 6: Net-(U11-FB) -> Net-(JP6-C)
Routing:
- net Net-(JP6-C): track 0.00 -> 34.8 mm, vias 0 -> 3
- net Net-(U11-FB): track 29.6 -> 0.00 mm, vias 2 -> 0
- net /misc/R_fb_24: track 0.00 -> 4.67 mm, vias 0 -> 1
- net /misc/R_fb_12: track 0.00 -> 4.48 mm, vias 0 -> 1
- net /+5v: track 501.0 -> 498.6 mm
- net GND: track 399.0 -> 398.1 mm
Other:
- board text added: "+ -"
- board text added: "-- 1.8v"
- board text added: "12V"
- board text added: "24V"
- board text added: "3.3v --"
- board text added: "JLCJLCJLCJLC"
- board text added: "Set GPIO Reference Voltage"
- board text added: "Set Vreg voltage"
- board text added: "Vin 12-48V DC"
- board text removed: "WayWayWay"
