File: duet_pi.kicad_pcb (KiCad board)
At the start: 4 copper layers, 134 x 140 mm, 120 parts, among them J1 USB_C_Receptacle_USB2.0, J10 690-019-298-412, J11 USB3_A, J12 THD-02-R, J13 Conn_01x22_Female, J14 690-019-298-412, J15 Bus_M.2_Socket_M, J16 Screw_Terminal_01x10, J2 THD-20-R, J4 THD-20-R, J5 Micro_SD_Card_Det, J6 Conn_01x03, J8 Conn_02x07_Odd_Even, J9 Conn_01x22_Female, M6 Fan, SW1 Right angle Tact button, U1 TPD4EUSB30, U10 TPP60508, U11 TPP60508, U2 TPD4EUSB30, U3 MagJack-A70-112-331N126, U4 74LVC1G07SE-7, U5 RT9742GGJ5, U6 RT9742SNGV, U7 AP22653W6, U8 ASEK-32.768KHZ-L-R-T, U9 AP3441SHE-7B

Commit message: incremental updates
Routing:
- net /CM5_HighSpeed/DPHY1_C_P: track 33.4 -> 33.9 mm
- net GND: vias 146 -> 159
- added copper zone on B.Cu, net GND
- added copper zone on F.Cu, net GND

Commit message: initial production
Parts:
- added J20: JST_SHBM04B-SRSS-TB, Connector_JST:JST_SH_BM04B-SRSS-TB_1x04-1MP_P1.00mm_Vertical, F.Cu at (66.6, 102.0)
- added J3: THD-02-R, Connector_PinHeader_2.54mm:PinHeader_2x02_P2.54mm_Vertical, F.Cu at (33.5, 55.9)
- added JP7: SolderJumper_3_Bridged12, Jumper:SolderJumper-3_P1.3mm_Bridged12_RoundedPad1.0x1.5mm, B.Cu at (68.6, 97.8)
- added JP8: SolderJumper_3_Bridged12, Jumper:SolderJumper-3_P1.3mm_Bridged12_RoundedPad1.0x1.5mm, B.Cu at (63.9, 98.0)
- added JP9: SolderJumper_2_Open, Jumper:SolderJumper-2_P1.3mm_Open_TrianglePad1.0x1.5mm, B.Cu at (68.4, 160.4)
- added TP4: TestPoint, TestPoint:TestPoint_Pad_D1.5mm, F.Cu at (117.8, 110.2)
- added TP5: TestPoint, TestPoint:TestPoint_Pad_D1.5mm, F.Cu at (132.8, 77.1)
- added TP6: TestPoint, TestPoint:TestPoint_Pad_D1.5mm, F.Cu at (41.5, 148.2)
- J14: value 690-019-298-412 -> WM1282DKR-ND
- J4: value THD-20-R -> THD-13-R
- moved J6 7.74 mm to (145.8, 172.8), turned to -90 degrees
- moved R6 7.47 mm to (125.3, 161.8)
- moved R7 6.77 mm to (128.8, 161.8)
- moved R3 4.83 mm to (29.4, 60.2), turned to 180 degrees
Connections:
- C1 pad 1: /+5v -> Net-(JP9-A)
- C2 pad 1: /+5v -> Net-(JP9-A)
- J1 pad A4: /+5v -> Net-(JP9-A)
- J1 pad A9: /+5v -> Net-(JP9-A)
- J1 pad B4: /+5v -> Net-(JP9-A)
- J1 pad B9: /+5v -> Net-(JP9-A)
- J7 pad 2: /CM5_GPIO ( Ethernet, GPIO, SDCARD)/PWM -> Net-(J7-Pin_2)
- J7 pad 4: /CM5_GPIO ( Ethernet, GPIO, SDCARD)/TACHO -> Net-(J7-Pin_4)
- R1 pad 1: /+5v -> Net-(JP9-A)
Routing:
- net /CM5_GPIO ( Ethernet, GPIO, SDCARD)/TR3_TAP: track 0.00 -> 56.9 mm
- net /CM5_HighSpeed/USB3-0-TX_N: track 48.3 -> 70.8 mm
- net /CM5_HighSpeed/USB3-0-TX_P: track 48.3 -> 70.8 mm
- net /CM5_GPIO ( Ethernet, GPIO, SDCARD)/TR2_TAP: track 0.00 -> 22.2 mm
- net Net-(JP9-A): track 0.00 -> 21.5 mm, vias 0 -> 2
- net /CM5_GPIO ( Ethernet, GPIO, SDCARD)/TR0_TAP: track 0.00 -> 17.6 mm
- net /CM5_GPIO ( Ethernet, GPIO, SDCARD)/TR1_TAP: track 0.00 -> 16.5 mm
- net /CM5_HighSpeed/USB3-1-RX_N: track 54.7 -> 70.0 mm
- net /CM5_HighSpeed/USB3-1-RX_P: track 57.2 -> 72.4 mm
- net /CM5_HighSpeed/USB3-0-D_N: track 57.1 -> 71.0 mm
- net /CM5_HighSpeed/USB3-0-D_P: track 57.2 -> 71.0 mm
- net /CM5_GPIO ( Ethernet, GPIO, SDCARD)/TRD3_N: track 86.7 -> 98.4 mm
- net /CM5_GPIO ( Ethernet, GPIO, SDCARD)/TRD3_P: track 86.6 -> 98.3 mm
- net /CM5_HighSpeed/DPHY0_D0_N: track 50.1 -> 59.8 mm
- net /CM5_HighSpeed/DPHY0_D0_P: track 50.1 -> 59.8 mm
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- removed copper zone on B.Cu, net GND
- removed copper zone on F.Cu, net GND
Other:
- board text added: "CAM/DISP0"
- board text added: "CAM/DISP1"
- board text added: "Ethernet"
- board text added: "Fit two jumpers for CAM/DISP 1"
- board text added: "HDMI 0"
- board text added: "HDMI1"
- board text added: "JST"
- board text added: "Molex KK"
- board text added: "PWM"
- board text added: "SD Card"
- board text added: "Tach"
- board text added: "USB 3.0"
- board text added: "USB Type-C 2.0"
- board text added: "USB Type-C Vbus connection. Avoid powering Duet Pi from two 5V sources"

Commit message: publish
Other:
- board text added: "Designed by Tim Eggebroten Released under CERN-OHL-S v2 license terms. Source available at https://github.com/taegge"
Changed lines of the file:
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@@
+		)
+	)
+	(gr_text "Designed by Tim Eggebroten\nReleased under CERN-OHL-S v2 license terms.\nSource available at https://github.com/taegge"
+		(at 152.67 83.49 270)
+		(layer "B.SilkS")
+		(effects
+			(font
+				(size 1 1)
+				(thickness 0.1)
+			)
+			(justify left bottom mirror)
 		)
 	)
