File: CM5_GPIO.kicad_sch (KiCad schematic)
At the start: 26 parts, among them J10 JST_SHBM04B-SRSS-TB, J11 THD-20-R, J12 THD-02-R, J13 Micro_SD_Card_Det, J8 Conn_02x07_Odd_Even, J9 Conn_01x03, SW1 Right angle Tact button, U3 74LVC1G07SE-7, U4 TPD4EUSB30, U5 TPD4EUSB30, U6 RT9742GGJ5, U7 MagJack-A70-112-331N126

Commit message: complete schematic
Parts:
- added J16: THD-20-R, Connector_IDC:IDC-Header_2x13_P2.54mm_Vertical, symbol Connector_Generic:Conn_02x20_Odd_Even
- BT1: digikey (none) -> 36-3034-ND
- C10: footprint Capacitor_SMD:C_0402_1005Metric -> Capacitor_SMD:C_0805_2012Metric_Pad1.18x1.45mm_HandSolder; digikey (none) -> 1276-1003-1-ND
- C9: footprint Capacitor_SMD:C_0805_2012Metric -> Capacitor_SMD:C_0805_2012Metric_Pad1.18x1.45mm_HandSolder; digikey (none) -> 1276-1096-1-ND
- D1: digikey (none) -> LTST-S270KGKT
- D2: digikey (none) -> LTST-S270KRKT
- J12: now not fitted
Connections:
- net +3.3v: now also J16.1 (Pin_1), J16.17 (Pin_17)
- net +5v: now also J16.2 (Pin_2), J16.4 (Pin_4)
- net GND: now also J16.14 (Pin_14), J16.20 (Pin_20), J16.25 (Pin_25), J16.6 (Pin_6), J16.9 (Pin_9)
- net GPIO10: now also J16.19 (Pin_19)
- net GPIO11: now also J16.23 (Pin_23)
- net GPIO14: now also J16.8 (Pin_8)
- net GPIO15: now also J16.10 (Pin_10)
- net GPIO17: now also J16.11 (Pin_11)
- net GPIO18: now also J16.12 (Pin_12)
- net GPIO2: now also J16.3 (Pin_3)
- net GPIO22: now also J16.15 (Pin_15)
- net GPIO23: now also J16.16 (Pin_16)
- net GPIO24: now also J16.18 (Pin_18)
- net GPIO25: now also J16.22 (Pin_22)
- net GPIO27: now also J16.13 (Pin_13)
- net GPIO3: now also J16.5 (Pin_5)
- net GPIO4: now also J16.7 (Pin_7)
- net GPIO7: now also J16.26 (Pin_26)
- net GPIO8: now also J16.24 (Pin_24)
- net GPIO9: now also J16.21 (Pin_21)
Other:
- note added: "26Way GPIO Header"
- moved on the sheet: D2, R7, R8, R9, TP2, U3

Commit message: stalled routing
Parts:
- removed R7: 0R, Resistor_SMD:R_0805_2012Metric_Pad1.20x1.40mm_HandSolder, symbol Device:R
- removed R8: nf, Resistor_SMD:R_0805_2012Metric_Pad1.20x1.40mm_HandSolder, symbol Device:R
- added JP1: SolderJumper_3_Bridged12, Jumper:SolderJumper-3_P1.3mm_Bridged12_RoundedPad1.0x1.5mm, symbol Jumper:SolderJumper_3_Bridged12
- J7: renamed from J10; value JST_SHBM04B-SRSS-TB -> (none); footprint Connector_JST:JST_SH_BM04B-SRSS-TB_1x04-1MP_P1.00mm_Vertical -> Connector:FanPinHeader_1x04_P2.54mm_Vertical; Field5 SHBM04B-SRSS-TB -> (none); Field6 SHBM04B-SRSS-TB -> (none)
- R2: renamed from R6; footprint Resistor_SMD:R_0402_1005Metric -> Resistor_SMD:R_0805_2012Metric_Pad1.20x1.40mm_HandSolder
- R3: renamed from R10; footprint Resistor_SMD:R_0402_1005Metric -> Resistor_SMD:R_0805_2012Metric_Pad1.20x1.40mm_HandSolder
- R4: renamed from R11; footprint Resistor_SMD:R_0402_1005Metric -> Resistor_SMD:R_0805_2012Metric_Pad1.20x1.40mm_HandSolder
- R5: renamed from R9; footprint Resistor_SMD:R_0402_1005Metric -> Resistor_SMD:R_0805_2012Metric_Pad1.20x1.40mm_HandSolder
- renumbered C10 to C3, C9 to C4, J11 to J2, J12 to J3, J16 to J4, J13 to J5, J9 to J6, U4 to U1, U5 to U2, U7 to U3, U3 to U4, U6 to U5
Connections:
- net +1.8v: now also JP1.3 (B)
- net +3.3v: now also JP1.1 (A)
- net GPIO_VREF: now also JP1.2 (C)

Commit message: pre-revise 5v route
Parts:
- J7: value (none) -> ~
Changed lines of the file:
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@@
 			)
 		)
-		(property "Value" ""
+		(property "Value" "~"
 			(at 146.05 183.515 0)
 			(effects

Commit message: incremental updates
Parts:
- BT1: digikey 36-3034-ND -> 36-3034-ND
- SW1: digikey (none) -> PTS645VL58-2 LFS
- U1, U2: digikey (none) -> 296-28063-1-ND
- U4: digikey (none) -> 74LVC1G07SE-7DICT-ND
- U5: digikey (none) -> 1028-1436-1-ND
Changed lines of the file:
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@@
 			)
 		)
+		(property "digikey" "296-28063-1-ND"
+			(at 203.2 33.02 0)
+			(effects
+				(font
+					(size 1.27 1.27)
+				)
+				(hide yes)
+			)
+		)
 		(pin "1"
 		)
@@
 			)
 		)
-		(property "digikey" "	\n36-3034-ND"
+		(property "digikey" "36-3034-ND"
 			(at 107.95 179.07 0)
 			(effects
@@
 			)
 		)
+		(property "digikey" "1028-1436-1-ND"
+			(at 248.92 163.83 0)
+			(effects
+				(font
+					(size 1.27 1.27)
+				)
+				(hide yes)
+			)
+		)
 		(pin "1"
 		)
@@
 			)
 		)
+		(property "digikey" "296-28063-1-ND"
+			(at 203.2 64.77 0)
+			(effects
+				(font
+					(size 1.27 1.27)
+				)
+				(hide yes)
+			)
+		)
 		(pin "1"
 		)
@@
 			)
 		)
+		(property "digikey" "PTS645VL58-2 LFS"
+			(at 76.2 177.8 0)
+			(effects
+				(font
+					(size 1.27 1.27)
+				)
+				(hide yes)
+			)
+		)
 		(pin "1"
 		)
@@
 			(at 180.34 149.86 0)
 			(effects
+				(font
+					(size 1.27 1.27)
+				)
+				(hide yes)
+			)
+		)
+		(property "digikey" "74LVC1G07SE-7DICT-ND"
+			(at 180.34 149.86 0)
+			(effects

Commit message: initial production
Parts:
- added J20: JST_SHBM04B-SRSS-TB, Connector_JST:JST_SH_BM04B-SRSS-TB_1x04-1MP_P1.00mm_Vertical, symbol Connector_Generic:Conn_01x04
- added JP7, JP8: SolderJumper_3_Bridged12, Jumper:SolderJumper-3_P1.3mm_Bridged12_RoundedPad1.0x1.5mm, symbol Jumper:SolderJumper_3_Bridged12
- J2: now not fitted
- J4: value THD-20-R -> THD-13-R
- J5: digikey (none) -> 2073-MEM2080-00-128-00-ADKR-ND
Connections:
- net +5v: now also J20.1 (Pin_1)
- net GND: now also J20.3 (Pin_3)
- net PWM: now also JP7.2 (C); no longer J7.2 (Pin_2)
- net TACHO: now also JP8.2 (C); no longer J7.4 (Pin_4)
- new net: J20.2 (Pin_2), JP7.1 (A)
- new net: J20.4 (Pin_4), JP8.1 (A)
- new net: J7.4 (Pin_4), JP8.3 (B)
- new net: J7.2 (Pin_2), JP7.3 (B)
Other:
- moved on the sheet: BT1, J7

Commit message: v0.1 prototype definition
Parts:
- J20: digikey (none) -> 455-BM04B-SRSS-TBCT-ND
- J4: digikey (none) -> SBH11-PBPC-D13-ST-BK
- J8: digikey (none) -> 2057-PH2-14-UA-ND
- Module1: digikey (none) -> 2x 10164227-1001A1RLF
- R2, R5: digikey (none) -> 311-1.00KCRCT-ND
- R3, R4: digikey (none) -> 311-470CRCT-ND
- U3: digikey (none) -> 535-14155-ND
Changed lines of the file:
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@@
 			)
 		)
+		(property "digikey" "311-470CRCT-ND"
+			(at 228.6 82.55 0)
+			(effects
+				(font
+					(size 1.27 1.27)
+				)
+				(hide yes)
+			)
+		)
 		(pin "1"
 		)
@@
 			)
 		)
+		(property "digikey" "311-1.00KCRCT-ND"
+			(at 187.96 139.7 0)
+			(effects
+				(font
+					(size 1.27 1.27)
+				)
+				(hide yes)
+			)
+		)
 		(pin "1"
 		)
@@
 			)
 		)
+		(property "digikey" "455-BM04B-SRSS-TBCT-ND"
+			(at 119.38 177.8 0)
+			(effects
+				(font
+					(size 1.27 1.27)
+				)
+				(hide yes)
+			)
+		)
 		(pin "1"
 		)
@@
 			)
 		)
+		(property "digikey" "535-14155-ND"
+			(at 264.16 95.25 0)
+			(effects
+				(font
+					(size 1.27 1.27)
+				)
+				(hide yes)
+			)
+		)
 		(pin "1"
 		)
@@
 			)
 		)
+		(property "digikey" "2057-PH2-14-UA-ND"
+			(at 33.02 180.34 0)
+			(effects
+				(font
+					(size 1.27 1.27)
+				)
+				(hide yes)
+			)
+		)
 		(pin "1"
 		)
@@
 			)
 		)
+		(property "digikey" "2x 10164227-1001A1RLF"
+			(at 68.58 80.01 0)
+			(effects
+				(font
+					(size 1.27 1.27)
+				)
+				(hide yes)
+			)
+		)
 		(pin "1"
 		)
@@
 			)
 		)
+		(property "digikey" "SBH11-PBPC-D13-ST-BK"
+			(at 153.67 118.11 0)
+			(effects
+				(font
+					(size 1.27 1.27)
+				)
+				(hide yes)
+			)
+		)
 		(pin "1"
 		)
@@
 			)
 		)
+		(property "digikey" "311-470CRCT-ND"
+			(at 228.6 77.47 0)
+			(effects
+				(font
+					(size 1.27 1.27)
+				)
+				(hide yes)
+			)
+		)
 		(pin "1"
 		)
@@
 			(at 113.03 43.18 0)
 			(effects
+				(font
+					(size 1.27 1.27)
+				)
+				(hide yes)
+			)
+		)
+		(property "digikey" "311-1.00KCRCT-ND"
+			(at 113.03 43.18 0)
+			(effects
