File: CM5_HighSpeed.kicad_sch (KiCad schematic)
At the start: 19 parts, among them J2 Conn_01x22_Female, J3 Conn_01x22_Female, J4 THD-02-R, J5 USB3_A, J6 690-019-298-412, J7 690-019-298-412, U1 AP22653W6, U2 RT9742SNGV

Commit message: complete schematic
Parts:
- C3, C5, C6: footprint Capacitor_SMD:C_0805_2012Metric -> Capacitor_SMD:C_0805_2012Metric_Pad1.18x1.45mm_HandSolder; digikey (none) -> 1276-1096-1-ND
- C4: digikey (none) -> 718-1100-1-ND
- C7, C8: footprint Capacitor_SMD:C_0402_1005Metric -> Capacitor_SMD:C_0805_2012Metric_Pad1.18x1.45mm_HandSolder; digikey (none) -> 1276-1003-1-ND
- J2, J3: digikey (none) -> HFJ122CT-ND
- J4: now not fitted
Changed lines of the file:
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@@
 			)
 		)
-		(property "Footprint" "Capacitor_SMD:C_0805_2012Metric"
+		(property "Footprint" "Capacitor_SMD:C_0805_2012Metric_Pad1.18x1.45mm_HandSolder"
 			(at 102.5652 186.69 0)
 			(effects
@@
 			)
 		)
-		(property "Datasheet" "https://search.murata.co.jp/Ceramy/image/img/A01X/G101/ENG/GRM21BR71A106KA73-01.pdf"
+		(property "Datasheet" ""
 			(at 101.6 182.88 0)
 			(effects
@@
 			)
 		)
+		(property "digikey" "1276-1096-1-ND "
+			(at 101.6 182.88 0)
+			(effects
+				(font
+					(size 1.27 1.27)
+				)
+				(hide yes)
+			)
+		)
 		(pin "1"
 		)
@@
 		(in_bom yes)
 		(on_board yes)
-		(dnp no)
+		(dnp yes)
 		(property "Reference" "J4"
 			(at 195.453 115.443 0)
@@
 			)
 		)
-		(property "Footprint" "Capacitor_SMD:C_0805_2012Metric"
+		(property "Footprint" "Capacitor_SMD:C_0805_2012Metric_Pad1.18x1.45mm_HandSolder"
 			(at 31.4452 185.42 0)
 			(effects
@@
 			)
 		)
-		(property "Datasheet" "https://search.murata.co.jp/Ceramy/image/img/A01X/G101/ENG/GRM21BR71A106KA73-01.pdf"
+		(property "Datasheet" ""
 			(at 30.48 181.61 0)
 			(effects
@@
 			)
 		)
+		(property "digikey" "1276-1096-1-ND "
+			(at 30.48 181.61 0)
+			(effects
+				(font
+					(size 1.27 1.27)
+				)
+				(hide yes)
+			)
+		)
 		(pin "1"
 		)
@@
 			)
 		)
-		(property "Footprint" "Capacitor_SMD:C_0402_1005Metric"
+		(property "Footprint" "Capacitor_SMD:C_0805_2012Metric_Pad1.18x1.45mm_HandSolder"
 			(at 199.0852 156.21 0)
 			(effects
@@
 			)
 		)
-		(property "Datasheet" "https://search.murata.co.jp/Ceramy/image/img/A01X/G101/ENG/GRM155R71C104KA88-01.pdf"
+		(property "Datasheet" ""
 			(at 198.12 152.4 0)
 			(effects
@@
 			)
 		)
+		(property "digikey" "1276-1003-1-ND"
+			(at 198.12 152.4 0)
+			(effects
+				(font
+					(size 1.27 1.27)
+				)
+				(hide yes)
+			)
+		)
 		(pin "1"
 		)
@@
 			)
 		)
-		(property "Footprint" "Capacitor_SMD:C_0805_2012Metric"
+		(property "Footprint" "Capacitor_SMD:C_0805_2012Metric_Pad1.18x1.45mm_HandSolder"
 			(at 112.7252 186.69 0)
 			(effects
@@
 			)
 		)
-		(property "Datasheet" "https://search.murata.co.jp/Ceramy/image/img/A01X/G101/ENG/GRM21BR71A106KA73-01.pdf"
+		(property "Datasheet" ""
 			(at 111.76 182.88 0)
 			(effects
@@
 			)
 		)
+		(property "digikey" "1276-1096-1-ND "
+			(at 111.76 182.88 0)
+			(effects
+				(font
+					(size 1.27 1.27)
+				)
+				(hide yes)
+			)
+		)
 		(pin "1"
 		)
@@
 			)
 		)
+		(property "digikey" "HFJ122CT-ND"
+			(at 157.48 123.19 0)
+			(effects
+				(font
+					(size 1.27 1.27)
+				)
+				(hide yes)
+			)
+		)
 		(pin "1"
 		)
@@
 			)
 		)
-		(property "Footprint" "Capacitor_SMD:C_0402_1005Metric"
+		(property "Footprint" "Capacitor_SMD:C_0805_2012Metric_Pad1.18x1.45mm_HandSolder"
 			(at 232.1052 156.21 0)
 			(effects
@@
 			)
 		)
-		(property "Datasheet" "https://search.murata.co.jp/Ceramy/image/img/A01X/G101/ENG/GRM155R71C104KA88-01.pdf"
+		(property "Datasheet" ""
 			(at 231.14 152.4 0)
 			(effects
@@
 			)
 		)
+		(property "digikey" "1276-1003-1-ND"
+			(at 231.14 152.4 0)
+			(effects
+				(font
+					(size 1.27 1.27)
+				)
+				(hide yes)
+			)
+		)
 		(pin "1"
 		)
@@
 			)
 		)
+		(property "digikey" "718-1100-1-ND"
+			(at 88.9 182.88 0)
+			(effects
+				(font
+					(size 1.27 1.27)
+				)
+				(hide yes)
+			)
+		)
 		(pin "1"
 		)
@@
 			(at 157.48 52.07 0)
 			(effects
+				(font
+					(size 1.27 1.27)
+				)
+				(hide yes)
+			)
+		)
+		(property "digikey" "HFJ122CT-ND"
+			(at 157.48 52.07 0)
+			(effects

Commit message: stalled routing
Parts:
- R6: renamed from R4; footprint Resistor_SMD:R_0402_1005Metric -> Resistor_SMD:R_0805_2012Metric_Pad1.20x1.40mm_HandSolder
- R7: renamed from R5; footprint Resistor_SMD:R_0402_1005Metric -> Resistor_SMD:R_0805_2012Metric_Pad1.20x1.40mm_HandSolder
- R8: renamed from R3; footprint Resistor_SMD:R_0402_1005Metric -> Resistor_SMD:R_0805_2012Metric_Pad1.20x1.40mm_HandSolder
- R9: renamed from R2; footprint Resistor_SMD:R_0402_1005Metric -> Resistor_SMD:R_0805_2012Metric_Pad1.20x1.40mm_HandSolder
- renumbered C6 to C10, C7 to C5, C8 to C6, C3 to C7, C4 to C8, C5 to C9, J6 to J10, J5 to J11, J4 to J12, J3 to J13, J7 to J14, J2 to J9, U2 to U6, U1 to U7

Commit message: nearing final routing
Parts:
- J14: footprint CM5IO:EDAC 690-019-298-412 -> Connector_Video:HDMI_Micro-D_Molex_46765-1x01; Field4 Farnell -> (none); Field5 2614936 -> (none); Field6 690-019-298-412 -> (none); Field7 EDAC -> (none); Field8 UCON00802 -> (none); Part Description HDMI Connector, Right Angle, 19 Contacts, Receptacle, Surfa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 -> (none); digikey (none) -> WM1282DKR-ND
Changed lines of the file:
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@@
 			)
 		)
-		(property "Footprint" "CM5IO:EDAC 690-019-298-412"
+		(property "Footprint" "Connector_Video:HDMI_Micro-D_Molex_46765-1x01"
 			(at 266.065 124.46 0)
 			(effects
@@
 			)
 		)
-		(property "Datasheet" "https://www.tme.eu/Document/f15dffbcfad8545e17826f72d36911c8/206A-SEAN-R03.pdf"
+		(property "Datasheet" ""
 			(at 266.065 124.46 0)
 			(effects
@@
 			)
 		)
-		(property "Field4" "Farnell"
+		(property "digikey" "WM1282DKR-ND"
 			(at 265.43 124.46 0)
 			(effects
-				(font
-					(size 1.27 1.27)
-				)
-				(hide yes)
-			)
-		)
-		(property "Field5" "2614936"
-			(at 265.43 124.46 0)
-			(effects
-				(font
-					(size 1.27 1.27)
-				)
-				(hide yes)
-			)
-		)
-		(property "Field6" "690-019-298-412"
-			(at 265.43 124.46 0)
-			(effects
-				(font
-					(size 1.27 1.27)
-				)
-				(hide yes)
-			)
-		)
-		(property "Field7" "EDAC"
-			(at 265.43 124.46 0)
-			(effects
-				(font
-					(size 1.27 1.27)
-				)
-				(hide yes)
-			)
-		)
-		(property "Part Description" "HDMI Connector, Right Angle, 19 Contacts, Receptacle, Surface Mount, Surface Mount Right Angle"
-			(at 265.43 124.46 0)
-			(effects
-				(font
-					(size 1.27 1.27)
-				)
-				(hide yes)
-			)
-		)
-		(property "Field8" "UCON00802"
-			(at 265.43 124.46 0)
-			(effects

Commit message: incremental updates
Parts:
- J14: value 690-019-298-412 -> WM1282DKR-ND
- U6: digikey (none) -> 1028-RT9742SNGVCT-ND
- U7: digikey (none) -> 31-AP22653W6-7CT-ND
Changed lines of the file:
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@@
 			)
 		)
+		(property "digikey" "31-AP22653W6-7CT-ND"
+			(at 60.96 179.07 0)
+			(effects
+				(font
+					(size 1.27 1.27)
+				)
+				(hide yes)
+			)
+		)
 		(pin "1"
 		)
@@
 			)
 		)
+		(property "digikey" "1028-RT9742SNGVCT-ND"
+			(at 214.63 152.4 0)
+			(effects
+				(font
+					(size 1.27 1.27)
+				)
+				(hide yes)
+			)
+		)
 		(pin "1"
 		)
@@
 			)
 		)
-		(property "Value" "690-019-298-412"
+		(property "Value" "WM1282DKR-ND"
 			(at 262.89 156.21 0)
 			(effects

Commit message: v0.1 prototype definition
Parts:
- J10: Field4 Farnell -> (none); Field5 2614936 -> (none); Field6 690-019-298-412 -> (none); Field7 EDAC -> (none); Field8 UCON00802 -> (none); digikey (none) -> 137-RAHHD19CT-ND
- J11: digikey (none) -> 380-1411-ND
- Module1: digikey (none) -> 2x 10164227-1001A1RLF
- R6, R7, R8: digikey (none) -> 311-2.20KCRCT-ND
- R9: digikey (none) -> 311-15.0KCRCT-ND
Changed lines of the file:
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@@
+			)
+		)
+		(property "digikey" "380-1411-ND"
+			(at 209.55 53.34 0)
+			(effects
+				(font
+					(size 1.27 1.27)
+				)
+				(hide yes)
 			)
 		)
@@
 			)
 		)
+		(property "digikey" "311-2.20KCRCT-ND"
+			(at 208.28 111.76 0)
+			(effects
+				(font
+					(size 1.27 1.27)
+				)
+				(hide yes)
+			)
+		)
 		(pin "1"
 		)
@@
 			)
 		)
+		(property "digikey" "311-2.20KCRCT-ND"
+			(at 215.9 111.76 0)
+			(effects
+				(font
+					(size 1.27 1.27)
+				)
+				(hide yes)
+			)
+		)
 		(pin "1"
 		)
@@
 			)
 		)
+		(property "digikey" "311-2.20KCRCT-ND"
+			(at 139.7 138.43 0)
+			(effects
+				(font
+					(size 1.27 1.27)
+				)
+				(hide yes)
+			)
+		)
 		(pin "1"
 		)
@@
 			)
 		)
+		(property "digikey" "2x 10164227-1001A1RLF"
+			(at -69.85 87.63 0)
+			(effects
+				(font
+					(size 1.27 1.27)
+				)
+				(hide yes)
+			)
+		)
 		(pin "1"
 		)
@@
 			)
 		)
+		(property "digikey" "311-15.0KCRCT-ND"
+			(at 80.01 179.07 0)
+			(effects
+				(font
+					(size 1.27 1.27)
+				)
+				(hide yes)
+			)
+		)
 		(pin "1"
 		)
@@
 			)
 		)
-		(property "Field4" "Farnell"
-			(at 265.43 52.07 0)
-			(effects
-				(font
-					(size 1.27 1.27)
-				)
-				(hide yes)
-			)
-		)
-		(property "Field5" "2614936"
-			(at 265.43 52.07 0)
-			(effects
-				(font
-					(size 1.27 1.27)
-				)
-				(hide yes)
-			)
-		)
-		(property "Field6" "690-019-298-412"
-			(at 265.43 52.07 0)
-			(effects
-				(font
-					(size 1.27 1.27)
-				)
-				(hide yes)
-			)
-		)
-		(property "Field7" "EDAC"
-			(at 265.43 52.07 0)
-			(effects
-				(font
-					(size 1.27 1.27)
-				)
-				(hide yes)
-			)
-		)
 		(property "Part Description" "HDMI Connector, Right Angle, 19 Contacts, Receptacle, Surface Mount, Surface Mount Right Angle"
 			(at 265.43 52.07 0)
@@
 			)
 		)
-		(property "Field8" "UCON00802"
+		(property "digikey" "137-RAHHD19CT-ND"
 			(at 265.43 52.07 0)
 			(effects
