File: PCIe-M2.kicad_sch (KiCad schematic)
At the start: 24 parts, among them J14 Bus_M.2_Socket_M, M1 M.2 Solder Nut, M2 M.2 Solder Nut, M3 M.2 Solder Nut, M4 M.2 Solder Nut, M5 M.2 Screw, U8 AP3441SHE-7B, U9 ASEK-32.768KHZ-L-R-T

Commit message: complete schematic
Parts:
- added M10, M7, M8, M9: M.2 Solder Nut, symbol CM5IO:SolderNut
- C11, C12, C15, C16, C17, C18: footprint Capacitor_SMD:C_0805_2012Metric -> Capacitor_SMD:C_0805_2012Metric_Pad1.18x1.45mm_HandSolder; digikey (none) -> 1276-1096-1-ND
- C13, C19: footprint Capacitor_SMD:C_0402_1005Metric -> Capacitor_SMD:C_0805_2012Metric_Pad1.18x1.45mm_HandSolder; digikey (none) -> 1276-1003-1-ND
- C14: footprint Capacitor_SMD:C_0402_1005Metric -> Capacitor_SMD:C_0805_2012Metric_Pad1.18x1.45mm_HandSolder; digikey (none) -> 1276-2525-1-ND
- D3: digikey (none) -> LTST-S270KGKT

Commit message: stalled routing
Parts:
- removed M10, M7, M8, M9: M.2 Solder Nut, symbol CM5IO:SolderNut
- R10: renamed from R15; footprint Resistor_SMD:R_0402_1005Metric -> Resistor_SMD:R_0805_2012Metric_Pad1.20x1.40mm_HandSolder
- R11: renamed from R13; footprint Resistor_SMD:R_0402_1005Metric -> Resistor_SMD:R_0805_2012Metric_Pad1.20x1.40mm_HandSolder
- R12: footprint Resistor_SMD:R_0402_1005Metric -> Resistor_SMD:R_0805_2012Metric_Pad1.20x1.40mm_HandSolder
- R13: renamed from R14; footprint Resistor_SMD:R_0402_1005Metric -> Resistor_SMD:R_0805_2012Metric_Pad1.20x1.40mm_HandSolder
- renumbered C19 to C11, C11 to C12, C12 to C13, C13 to C14, C14 to C15, C15 to C16, C16 to C17, C17 to C18, C18 to C19, J14 to J15, U9 to U8, U8 to U9

Commit message: incremental updates
Parts:
- U8: digikey (none) -> 535-ASEK-32.768KHZ-L-R-TCT-ND
- U9: digikey (none) -> AP3441SHE-7BDICT-ND
Changed lines of the file:
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@@
+			)
+		)
+		(property "digikey" "AP3441SHE-7BDICT-ND"
+			(at 66.04 173.99 0)
+			(effects
+				(font
+					(size 1.27 1.27)
+				)
+				(hide yes)
 			)
 		)
@@
 			(at 208.28 135.89 0)
 			(effects
+				(font
+					(size 1.27 1.27)
+				)
+				(hide yes)
+			)
+		)
+		(property "digikey" "535-ASEK-32.768KHZ-L-R-TCT-ND"
+			(at 208.28 135.89 0)
+			(effects

Commit message: initial production
Parts:
- added TP6: TestPoint, TestPoint:TestPoint_Pad_D1.5mm, symbol Connector:TestPoint
Connections:
- net M2_3v3: now also TP6.1
Changed lines of the file:
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@@
+	)
+	(symbol
+		(lib_id "Connector:TestPoint")
+		(at 144.78 173.99 0)
+		(unit 1)
+		(exclude_from_sim no)
+		(in_bom yes)
+		(on_board yes)
+		(dnp no)
+		(property "Reference" "TP6"
+			(at 135.128 169.164 0)
+			(effects
+				(font
+					(size 1.27 1.27)
+				)
+				(justify left)
+			)
+		)
+		(property "Value" "TestPoint"
+			(at 135.128 171.704 0)
+			(effects
+				(font
+					(size 1.27 1.27)
+				)
+				(justify left)
+			)
+		)
+		(property "Footprint" "TestPoint:TestPoint_Pad_D1.5mm"
+			(at 149.86 173.99 0)
+			(effects
+				(font
+					(size 1.27 1.27)
+				)
+				(hide yes)
+			)
+		)
+		(property "Datasheet" "~"
+			(at 149.86 173.99 0)
+			(effects
+				(font
+					(size 1.27 1.27)
+				)
+				(hide yes)
+			)
+		)
+		(property "Description" "test point"
+			(at 144.78 173.99 0)
+			(effects
+				(font
+					(size 1.27 1.27)
+				)
+				(hide yes)
+			)
+		)
+		(pin "1"
+		)
+		(instances
+			(project ""
+				(path "/c80e2680-7312-4906-8194-724a8268cfde/d7b8ce31-b426-4b84-8730-2ca9f82012ca"
+					(reference "TP6")
+					(unit 1)
+				)
+			)
+		)
 	)
 	(symbol

Commit message: v0.1 prototype definition
Parts:
- J15: digikey (none) -> 609-6590CT-ND
- L1: digikey (none) -> 118-SRP5030CC-2R2MCT-ND
- R10: digikey (none) -> 311-1.00KCRCT-ND
- R11: digikey (none) -> 13-RC0805FR-1310KLCT-ND
- R12: digikey (none) -> 311-100KCRCT-ND
- R13: digikey (none) -> 311-2.20KCRCT-ND
Changed lines of the file:
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@@
+			)
+		)
+		(property "digikey" "118-SRP5030CC-2R2MCT-ND"
+			(at 93.98 173.99 0)
+			(effects
+				(font
+					(size 1.27 1.27)
+				)
+				(hide yes)
 			)
 		)
@@
 			)
 		)
+		(property "digikey" "311-2.20KCRCT-ND"
+			(at 111.76 186.69 0)
+			(effects
+				(font
+					(size 1.27 1.27)
+				)
+				(hide yes)
+			)
+		)
 		(pin "1"
 		)
@@
 		)
 		(property "Part Description" "Resistor 10K M1005 1% 63mW"
+			(at 111.76 177.8 0)
+			(effects
+				(font
+					(size 1.27 1.27)
+				)
+				(hide yes)
+			)
+		)
+		(property "digikey" "13-RC0805FR-1310KLCT-ND"
 			(at 111.76 177.8 0)
 			(effects
@@
 			)
 		)
+		(property "digikey" "311-1.00KCRCT-ND"
+			(at 194.31 88.9 0)
+			(effects
+				(font
+					(size 1.27 1.27)
+				)
+				(hide yes)
+			)
+		)
 		(pin "1"
 		)
@@
 			)
 		)
+		(property "digikey" "311-100KCRCT-ND"
+			(at 81.28 180.34 0)
+			(effects
+				(font
+					(size 1.27 1.27)
+				)
+				(hide yes)
+			)
+		)
 		(pin "1"
 		)
@@
 			(at 153.67 86.36 0)
 			(effects
+				(font
+					(size 1.27 1.27)
+				)
+				(hide yes)
+			)
+		)
+		(property "digikey" "609-6590CT-ND"
+			(at 153.67 86.36 0)
+			(effects
