File: duet_pi.kicad_sch (KiCad schematic)
At the start: 4 parts

Commit message: CM5
Parts:
- removed H1, H2, H3, H4: MountingHole, MountingHole:MountingHole_4.3mm_M4, symbol Mechanical:MountingHole
- added C1, C2: 100n, Capacitor_SMD:C_0402_1005Metric, symbol Device:C
- added J1: USB_C_Receptacle_USB2.0, Connector_USB:USB_C_Receptacle_GCT_USB4105-xx-A_16P_TopMnt_Horizontal, symbol Connector:USB_C_Receptacle_USB2.0_16P
- added R1: 2.2K 1%, Resistor_SMD:R_0402_1005Metric, symbol Device:R
Connections:
- net +5v: now also C1.1, C2.1, J1.A4 (VBUS), J1.A9 (VBUS), J1.B4 (VBUS), J1.B9 (VBUS), R1.1
- new net CC1: J1.A5 (CC1)
- new net CC2: J1.B5 (CC2)
- new net GND: C1.2, C2.2, J1.A1 (GND), J1.A12 (GND), J1.B1 (GND), J1.B12 (GND), J1.S1 (SHIELD), R1.2
- new net USB2_N: J1.A7 (D-), J1.B7 (D-)
- new net USB2_P: J1.A6 (D+), J1.B6 (D+)
- no-connect marks 0 -> 2
Other:
- removed sheet CM4_GPIO ( Ethernet, GPIO, SDCARD)
- removed sheet CM4_HighSpeed
- removed sheet PSUs
- removed sheet RTC , Wakeup, FAN
- removed sheet USB2-HUB
- added sheet CM5_GPIO ( Ethernet, GPIO, SDCARD) (CM5_GPIO.kicad_sch)
- added sheet CM5_HighSpeed (CM5_HighSpeed.kicad_sch)
- added sheet PCIe-M2 (PCIe-M2.kicad_sch)
- added sheet misc (misc.kicad_sch)
- note added: "Connectors ------ M2 MKey"
- note added: "Connectors ------- Ethernet SDCARD 40way RPI Jumpers Fan Battery"
- note added: "Connectors ------- HDMI 0 HDMI 1 CSI/DSI 0 CSI/DSI 1"
- note added: "Discharge Resistor Needed by some Type C PSUs"
- note added: "TypeC Power connector"
- note removed: "Connectors ------- DC Barrel Jack 4 pin power"
- note removed: "Connectors ------- Dual USB microUSB"
- note removed: "Connectors ------- Ethernet SDCARD 40way RPI Jumpers"
- note removed: "Connectors ------- FAN Battery"
- note removed: "Connectors ------- HDMI 0 HDMI 1 CSI 0 CSI 1 DSI 0 DSI 1"
- company: © 2020-2022 Raspberry Pi Ltd (formerly Raspberry Pi (Trading) Ltd.) -> (none)
- title: Compute Module 4 IO Board - Top Level -> (none)

Commit message: complete schematic
Parts:
- C1, C2: footprint Capacitor_SMD:C_0402_1005Metric -> Capacitor_SMD:C_0805_2012Metric_Pad1.18x1.45mm_HandSolder; digikey (none) -> 1276-1003-1-ND
Other:
- sheet misc ports: added 5v; removed none
Changed lines of the file:
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@@
+	(wire
+		(pts
+			(xy 25.4 135.89) (xy 39.37 135.89)
+		)
+		(stroke
+			(width 0)
+			(type default)
+		)
+	)
 	(wire
 		(pts
@@
 	(label "CC1"
 		(at 121.92 137.16 0)
+		(fields_autoplaced yes)
+		(effects
+			(font
+				(size 1.27 1.27)
+			)
+			(justify left bottom)
+		)
+	)
+	(label "+5v"
+		(at 25.4 135.89 0)
 		(fields_autoplaced yes)
 		(effects
@@
 			)
 		)
-		(property "Footprint" "Capacitor_SMD:C_0402_1005Metric"
+		(property "Footprint" "Capacitor_SMD:C_0805_2012Metric_Pad1.18x1.45mm_HandSolder"
 			(at 75.8952 86.36 0)
 			(effects
@@
 			)
 		)
-		(property "Datasheet" "https://search.murata.co.jp/Ceramy/image/img/A01X/G101/ENG/GRM155R71C104KA88-01.pdf"
+		(property "Datasheet" ""
 			(at 74.93 82.55 0)
 			(effects
@@
 		)
 		(property "Part Description" "	0.1uF 10% 16V Ceramic Capacitor X7R 0402 (1005 Metric)"
+			(at 74.93 82.55 0)
+			(effects
+				(font
+					(size 1.27 1.27)
+				)
+				(hide yes)
+			)
+		)
+		(property "digikey" "1276-1003-1-ND"
 			(at 74.93 82.55 0)
 			(effects
@@
 			)
 		)
-		(property "Footprint" "Capacitor_SMD:C_0402_1005Metric"
+		(property "Footprint" "Capacitor_SMD:C_0805_2012Metric_Pad1.18x1.45mm_HandSolder"
 			(at 87.3252 86.36 0)
 			(effects
@@
 			)
 		)
-		(property "Datasheet" "https://search.murata.co.jp/Ceramy/image/img/A01X/G101/ENG/GRM155R71C104KA88-01.pdf"
+		(property "Datasheet" ""
 			(at 86.36 82.55 0)
 			(effects
@@
 		)
 		(property "Part Description" "	0.1uF 10% 16V Ceramic Capacitor X7R 0402 (1005 Metric)"
+			(at 86.36 82.55 0)
+			(effects
+				(font
+					(size 1.27 1.27)
+				)
+				(hide yes)
+			)
+		)
+		(property "digikey" "1276-1003-1-ND"
 			(at 86.36 82.55 0)
 			(effects
@@
 			)
 		)
+		(pin "5v" input
+			(at 39.37 135.89 180)
+			(effects
+				(font
+					(size 1.27 1.27)
+				)
+				(justify left)
+			)
+		)

Commit message: stalled routing
Parts:
- J1: Field5 USBF31-0171 -> (none); Field6 USBF31-0171 -> (none); Field7 MTCONN -> (none); digikey (none) -> 2073-USB4105-GF-ACT-ND
- R1: footprint Resistor_SMD:R_0402_1005Metric -> Resistor_SMD:R_0805_2012Metric_Pad1.20x1.40mm_HandSolder
Changed lines of the file:
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@@
 	(label "CC1"
 		(at 121.92 137.16 0)
-		(fields_autoplaced yes)
 		(effects
 			(font
@@
 	(label "+5v"
 		(at 25.4 135.89 0)
-		(fields_autoplaced yes)
 		(effects
 			(font
@@
 	(label "USB2_P"
 		(at 77.47 68.58 180)
-		(fields_autoplaced yes)
 		(effects
 			(font
@@
 	(label "+5v"
 		(at 74.93 78.74 0)
-		(fields_autoplaced yes)
 		(effects
 			(font
@@
 	(label "CC2"
 		(at 121.92 139.7 0)
-		(fields_autoplaced yes)
 		(effects
 			(font
@@
 	(label "CC1"
 		(at 67.31 55.88 0)
-		(fields_autoplaced yes)
 		(effects
 			(font
@@
 	(label "+3.3v"
 		(at 122.555 82.55 0)
-		(fields_autoplaced yes)
 		(effects
 			(font
@@
 	(label "USB2_N"
 		(at 77.47 63.5 180)
-		(fields_autoplaced yes)
 		(effects
 			(font
@@
 	(label "+5v"
 		(at 191.77 132.08 0)
-		(fields_autoplaced yes)
 		(effects
 			(font
@@
 	(label "+5v"
 		(at 248.92 71.12 0)
-		(fields_autoplaced yes)
 		(effects
 			(font
@@
 	(label "+5v"
 		(at 122.555 78.74 0)
-		(fields_autoplaced yes)
 		(effects
 			(font
@@
 	(label "CC2"
 		(at 67.31 58.42 0)
-		(fields_autoplaced yes)
 		(effects
 			(font
@@
 	(label "+5v"
 		(at 67.31 50.8 0)
-		(fields_autoplaced yes)
 		(effects
 			(font
@@
 	(label "+3.3v"
 		(at 191.77 137.16 0)
-		(fields_autoplaced yes)
 		(effects
 			(font
@@
 		(on_board yes)
 		(dnp no)
-		(property "Reference" "#PWR01"
+		(property "Reference" "#PWR03"
 			(at 45.72 96.52 0)
 			(effects
@@
 			(project "duet_pi"
 				(path "/c80e2680-7312-4906-8194-724a8268cfde"
-					(reference "#PWR01")
+					(reference "#PWR03")
 					(unit 1)
 				)
@@
 			)
 		)
-		(property "Field5" "USBF31-0171"
+		(property "Part Description" "USBC USB2 data and power connector"
 			(at 49.53 66.04 0)
 			(effects
@@
 			)
 		)
-		(property "Field6" "USBF31-0171"
-			(at 49.53 66.04 0)
-			(effects
-				(font
-					(size 1.27 1.27)
-				)
-				(hide yes)
-			)
-		)
-		(property "Field7" "MTCONN"
-			(at 49.53 66.04 0)
-			(effects
-				(font
-					(size 1.27 1.27)
-				)
-				(hide yes)
-			)
-		)
-		(property "Part Description" "USBC USB2 data and power connector"
+		(property "digikey" "2073-USB4105-GF-ACT-ND"
 			(at 49.53 66.04 0)
 			(effects
@@
 		(on_board yes)
 		(dnp no)
-		(property "Reference" "#PWR03"
+		(property "Reference" "#PWR01"
 			(at 90.17 64.77 0)
 			(effects
@@
 			(project "duet_pi"
 				(path "/c80e2680-7312-4906-8194-724a8268cfde"
-					(reference "#PWR03")
+					(reference "#PWR01")
 					(unit 1)
 				)
@@
 			)
 		)
-		(property "Footprint" "Resistor_SMD:R_0402_1005Metric"
+		(property "Footprint" "Resistor_SMD:R_0805_2012Metric_Pad1.20x1.40mm_HandSolder"
 			(at 88.392 54.61 90)
 			(effects

Commit message: initial production
Parts:
- added JP9: SolderJumper_2_Open, Jumper:SolderJumper-2_P1.3mm_Open_TrianglePad1.0x1.5mm, symbol Jumper:SolderJumper_2_Open
Connections:
- net +5v: now also JP9.2 (B); no longer C1.1, C2.1, J1.A4 (VBUS), J1.A9 (VBUS), J1.B4 (VBUS), J1.B9 (VBUS), R1.1
- new net: C1.1, C2.1, J1.A4 (VBUS), J1.A9 (VBUS), J1.B4 (VBUS), J1.B9 (VBUS), JP9.1 (A), R1.1
Changed lines of the file:
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@@
 	(paper "A4")
+	(junction
+		(at 66.04 50.8)
+		(diameter 0)
+		(color 0 0 0 0)
+	)
 	(junction
 		(at 64.77 68.58)
@@
 	)
 	(junction
+		(at 90.17 50.8)
+		(diameter 0)
+		(color 0 0 0 0)
+	)
+	(junction
 		(at 74.93 86.36)
 		(diameter 0)
 		(color 0 0 0 0)
 	)
+	(junction
+		(at 78.74 78.74)
+		(diameter 0)
+		(color 0 0 0 0)
+	)
 	(no_connect
 		(at 64.77 81.28)
@@
 	(wire
 		(pts
+			(xy 101.6 50.8) (xy 100.33 50.8)
+		)
+		(stroke
+			(width 0)
+			(type default)
+		)
+	)
+	(wire
+		(pts
 			(xy 165.1 102.87) (xy 165.1 118.11)
 		)
@@
 	(wire
 		(pts
-			(xy 74.93 78.74) (xy 86.36 78.74)
+			(xy 74.93 78.74) (xy 78.74 78.74)
+		)
+		(stroke
+			(width 0)
+			(type default)
+		)
+	)
+	(wire
+		(pts
+			(xy 66.04 50.8) (xy 90.17 50.8)
 		)
 		(stroke
@@
 	(wire
 		(pts
+			(xy 78.74 78.74) (xy 86.36 78.74)
+		)
+		(stroke
+			(width 0)
+			(type default)
+		)
+	)
+	(wire
+		(pts
 			(xy 115.57 54.61) (xy 115.57 68.58)
 		)
@@
 	(wire
 		(pts
+			(xy 90.17 50.8) (xy 92.71 50.8)
+		)
+		(stroke
+			(width 0)
+			(type default)
+		)
+	)
+	(wire
+		(pts
 			(xy 115.57 54.61) (xy 132.08 54.61)
 		)
@@
 	(wire
 		(pts
-			(xy 64.77 50.8) (xy 90.17 50.8)
+			(xy 64.77 50.8) (xy 66.04 50.8)
+		)
+		(stroke
+			(width 0)
+			(type default)
+		)
+	)
+	(wire
+		(pts
+			(xy 66.04 50.8) (xy 66.04 73.66)
 		)
 		(stroke
@@
 	(wire
 		(pts
+			(xy 66.04 73.66) (xy 78.74 73.66)
+		)
+		(stroke
+			(width 0)
+			(type default)
+		)
+	)
+	(wire
+		(pts
 			(xy 148.59 102.87) (xy 148.59 118.11)
 		)
@@
 		(pts
 			(xy 189.23 137.16) (xy 198.12 137.16)
+		)
+		(stroke
+			(width 0)
+			(type default)
+		)
+	)
+	(wire
+		(pts
+			(xy 78.74 73.66) (xy 78.74 78.74)
 		)
 		(stroke
@@
 		)
 	)
-	(label "+5v"
-		(at 74.93 78.74 0)
-		(effects
-			(font
-				(size 1.27 1.27)
-			)
-			(justify left bottom)
-		)
-	)
 	(label "CC2"
 		(at 121.92 139.7 0)
@@
 	)
 	(label "+5v"
-		(at 67.31 50.8 0)
+		(at 101.6 50.8 0)
 		(effects
 			(font
@@
 					(unit 1)
 				)
+			)
+		)
+	)
+	(symbol
+		(lib_id "Jumper:SolderJumper_2_Open")
+		(at 96.52 50.8 0)
+		(unit 1)
+		(exclude_from_sim yes)
+		(in_bom no)
+		(on_board yes)
+		(dnp no)
+		(property "Reference" "JP9"
+			(at 96.52 48.006 0)
+			(effects
+				(font
+					(size 1.27 1.27)
+				)
+			)
+		)
+		(property "Value" "SolderJumper_2_Open"
+			(at 96.52 46.99 0)
+			(effects
+				(font
+					(size 1.27 1.27)
+				)
+				(hide yes)
+			)
+		)
+		(property "Footprint" "Jumper:SolderJumper-2_P1.3mm_Open_TrianglePad1.0x1.5mm"
+			(at 102.108 33.528 0)
+			(effects
+				(font
+					(size 1.27 1.27)
+				)
+				(hide yes)
+			)
+		)
+		(property "Datasheet" "~"
+			(at 96.52 50.8 0)
+			(effects
+				(font
+					(size 1.27 1.27)
+				)
+				(hide yes)
+			)
+		)
+		(property "Description" "Solder Jumper, 2-pole, open"
+			(at 96.52 50.8 0)
+			(effects
+				(font
+					(size 1.27 1.27)
+				)
+				(hide yes)
+			)
+		)
+		(pin "2"
+		)
+		(pin "1"
+		)
+		(instances
+			(project ""
+				(path "/c80e2680-7312-4906-8194-724a8268cfde"
+					(reference "JP9")
+					(unit 1)
+				)

Commit message: v0.1 prototype definition
Parts:
- R1: digikey (none) -> 311-2.20KCRCT-ND
Changed lines of the file:
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@@
+			)
+		)
+		(property "digikey" "311-2.20KCRCT-ND"
+			(at 90.17 54.61 0)
+			(effects
+				(font
+					(size 1.27 1.27)
+				)
+				(hide yes)
 			)
 		)
