File: misc.kicad_sch (KiCad schematic)
At the start: 3 parts, among them J15 Conn_Coaxial

Commit message: complete schematic
Parts:
- removed AE1: Antenna_Chip, RF_Antenna:Abracon_PRO-OB-440, symbol Device:Antenna_Chip
- removed AE2: Antenna_Shield, RF_Antenna:Abracon_PRO-OB-440, symbol Device:Antenna_Shield
- added C20: 10uF, Capacitor_SMD:C_1210_3225Metric_Pad1.33x2.70mm_HandSolder, symbol Device:C
- added C21: 100n, Capacitor_SMD:C_0805_2012Metric_Pad1.18x1.45mm_HandSolder, symbol Device:C
- added C22: C, symbol Device:C
- added D4: D_Schottky, Diode_SMD:D_SMA_Handsoldering, symbol Device:D_Schottky
- added F1, F2, F3: MCCQ-122, footprints:MCCQ-122, symbol Device:Fuse
- added H1, H2, H3, H4: ~, MountingHole:MountingHole_4.3mm_M4, symbol Mechanical:MountingHole
- added J17: HB9500-9.5-8P, footprints:HB9500-9.5-8P, symbol Connector:Screw_Terminal_01x08
- added L2: 8.2uH, footprints:SMD_inductor_07A7, symbol Device:L
- added M6: Fan, footprints:fan_40mm_M3, symbol Motor:Fan
- added R16: 49.9k, symbol Device:R
- added R17: 100k, symbol Device:R
- added R18: 17.8k, symbol Device:R
- added U10: LV14360, footprints:LV14360, symbol symbols:LV14360
Connections:
- new net: C21.2, D4.1 (K), L2.1, U10.8 (SW)
- new net: R17.1, R18.2, U10.5 (FB)
- new net: C20.1, U10.6 (PGOOD)
- new net: R16.2, U10.4 (RT/SYNC)
- new net: C21.1, U10.1 (BOOT)
- new net: F3.1, J17.2 (Pin_2)
- new net: F2.1, J17.4 (Pin_4)
- new net: F1.1, J17.6 (Pin_6)
- new net 5v: C22.1, L2.2, R17.2
- new net GND: C20.2, C22.2, D4.2 (A), J17.1 (Pin_1), J17.3 (Pin_3), J17.5 (Pin_5), J17.7 (Pin_7), M6.1 (gnd), R16.1, R18.1, U10.7 (GND), U10.9 (thermal)
- new net Vin: F1.2, F2.2, F3.2, J17.8 (Pin_8), U10.2 (VIN), U10.3 (EN)

Commit message: stalled routing
Parts:
- removed J17: HB9500-9.5-8P, footprints:HB9500-9.5-8P, symbol Connector:Screw_Terminal_01x08
- removed U10: LV14360, footprints:LV14360, symbol symbols:LV14360
- added AE1: SR4W035, footprints:SR4W035, symbol Device:Antenna_Shield
- added C23, C34: 100n, Capacitor_SMD:C_0805_2012Metric_Pad1.18x1.45mm_HandSolder, symbol Device:C
- added C24, C25, C26, C31, C32, C35, C36, C37: 10uF, Capacitor_SMD:C_1210_3225Metric_Pad1.33x2.70mm_HandSolder, symbol Device:C
- added C27, C38: 10000pF, Capacitor_SMD:C_0805_2012Metric_Pad1.18x1.45mm_HandSolder, symbol Device:C
- added C28, C39: 47pF, Capacitor_SMD:C_0805_2012Metric_Pad1.18x1.45mm_HandSolder, symbol Device:C
- added C29, C40: 4.7nF, Capacitor_SMD:C_0805_2012Metric_Pad1.18x1.45mm_HandSolder, symbol Device:C
- added C30: C, Capacitor_SMD:C_0805_2012Metric, symbol Device:C
- added C33: 0.1uF, Capacitor_SMD:C_0805_2012Metric_Pad1.18x1.45mm_HandSolder, symbol Device:C
- added D5: D_Schottky, Diode_SMD:D_SMA_Handsoldering, symbol Device:D_Schottky
- added F4: MCCQ-122, footprints:MCCQ-122, symbol Device:Fuse
- added J16: Screw_Terminal_01x10, footprints:HB9500-9.5-10p, symbol Connector:Screw_Terminal_01x10
- added J18, J19: Conn_02x13_Odd_Even, symbol Connector_Generic:Conn_02x13_Odd_Even
- added JP2, JP3, JP4, JP5: SolderJumper_3_Open, footprints:resistor_jumper_3_way_0805, symbol Jumper:SolderJumper_3_Open
- added L3, L4: 2.2nH, Inductor_SMD:L_0805_2012Metric_Pad1.05x1.20mm_HandSolder, symbol Device:L
- added L5: 8.2uH, footprints:SMD_inductor_07A7, symbol Device:L
- added M10, M7, M8, M9: M3 Solder Nut, symbol CM5IO:SolderNut
- added R14, R15, R20, R21, R22: R, Resistor_SMD:R_0805_2012Metric_Pad1.20x1.40mm_HandSolder, symbol Device:R
- added R19, R25, R26: 3.24k, Resistor_SMD:R_0805_2012Metric_Pad1.20x1.40mm_HandSolder, symbol Device:R
- added R23: 100k, Resistor_SMD:R_0805_2012Metric_Pad1.20x1.40mm_HandSolder, symbol Device:R
- added R24: 240k, Resistor_SMD:R_0805_2012Metric_Pad1.20x1.40mm_HandSolder, symbol Device:R
- added U10, U11: TPP60508, footprints:DFN-10_EP_4x4_Pitch0.8mm, symbol symbols:TPP60508
- C20: now fitted
- C21: value 100n -> 10uF; footprint Capacitor_SMD:C_0805_2012Metric_Pad1.18x1.45mm_HandSolder -> Capacitor_SMD:C_1210_3225Metric_Pad1.33x2.70mm_HandSolder; digikey 1276-1003-1-ND -> 490-GRM32EC72A106ME05LCT-ND
- C22: value C -> 0.1uF; footprint (none) -> Capacitor_SMD:C_0805_2012Metric_Pad1.18x1.45mm_HandSolder
- J17: renamed from J15; footprint (none) -> Connector_Coaxial:U.FL_Hirose_U.FL-R-SMT-1_Vertical; digikey (none) -> H9161DKR-ND
- R16: value 49.9k -> 100k; footprint (none) -> Resistor_SMD:R_0805_2012Metric_Pad1.20x1.40mm_HandSolder; digikey (none) -> 311-100KCRDKR-ND
- R17: value 100k -> 240k; footprint (none) -> Resistor_SMD:R_0805_2012Metric_Pad1.20x1.40mm_HandSolder; digikey (none) -> 311-240KCRDKR-ND
- R18: value 17.8k -> 19.1k; footprint (none) -> Resistor_SMD:R_0805_2012Metric_Pad1.20x1.40mm_HandSolder; digikey (none) -> 311-19.1KCRDKR-ND
Connections:
- net 5v: now also R16.2, C24.1, C25.1, C26.1; no longer C22.1, R17.2
- net GND: now also C21.2, R17.1, C24.2, C25.2, C26.2, C27.2, C28.2, C29.2, C31.2, C32.2, C33.2, C35.2, C36.2, C37.2, C38.2, C39.2, C40.2, D5.2 (A), J16.1 (Pin_1), J16.3 (Pin_3), J16.5 (Pin_5), J16.7 (Pin_7), J16.9 (Pin_9), R15.2, R20.2, R22.2, R24.1, R25.1, U10.11 (therm), U10.8 (GND), U11.11 (therm), U11.8 (GND); no longer R16.1
- net Vin: now also C20.1, C21.1, C22.1, C31.1, C32.1, C33.1, J16.10 (Pin_10), JP2.1 (A), JP3.1 (A), JP4.1 (A), JP5.1 (A), R14.1, R21.1, U10.2 (VIN), U11.2 (VIN); no longer F1.2, F2.2, F3.2
- net at D4.1 (K), L2.1: now also C23.2, U10.9 (SW); no longer C21.2
- net at R18.2: now also R16.1, U10.6 (FB); no longer R17.1
- net at J17.1 (In): now also C30.2, L4.1
- net at J17.2 (Ext): now also AE1.3 (gnd), AE1.4 (gnd), AE1.6 (gnd), L3.2, L4.2, R20.1
- net at F3.1: now also J16.4 (Pin_4)
- net at F2.1: now also J16.6 (Pin_6)
- net at F1.1: now also J16.8 (Pin_8)
- new net: C23.1, U10.1 (BOOT)
- new net: F4.2, JP5.2 (C)
- new net: R17.2, U10.5 (RT/CLT)
- new net: R23.1, R25.2, U11.6 (FB)
- new net: F2.2, JP3.2 (C)
- new net: F4.1, J16.2 (Pin_2)
- new net: C34.1, U11.1 (BOOT)
- new net: R21.2, R22.1, U11.3 (EN)
- new net: C38.1, U11.4 (SS/TR)
- new net: R24.2, U11.5 (RT/CLT)
- new net: C39.1, R26.2, U11.7 (COMP)
- new net: C34.2, D5.1 (K), L5.1, U11.9 (SW)
- new net: AE1.2 (feed), C30.1, L3.1
- new net: F3.2, JP4.2 (C)
- new net: C40.1, R26.1
- new net: C27.1, U10.4 (SS/TR)
- new net: R14.2, R15.1, U10.3 (EN)
- new net: F1.2, JP2.2 (C)
- new net: C28.1, R19.2, U10.7 (COMP)
- new net: C29.1, R19.1
- new net Vreg2: C35.1, C36.1, C37.1, JP2.3 (B), JP3.3 (B), JP4.3 (B), JP5.3 (B), L5.2, R23.2
Other:
- moved on the sheet: F1, F2, F3, H1, H2, H3, H4, J17, M6

Commit message: pre-revise 5v route
Other:
- moved on the sheet: AE1, C30, J17, L3, L4, R20

Commit message: nearing final routing
Parts:
- added JP6: SolderJumper_3_Open, Jumper:SolderJumper-3_P1.3mm_Open_RoundedPad1.0x1.5mm, symbol Jumper:SolderJumper_3_Open
- added R27: 10.5k, Resistor_SMD:R_0805_2012Metric_Pad1.20x1.40mm_HandSolder, symbol Device:R
- R16, R23: value 100k -> 147k; digikey 311-100KCRDKR-ND -> 311-147KCRDKR-ND
- R18: value 19.1k -> 28k; digikey 311-19.1KCRDKR-ND -> 311-28.0KCRDKR-ND
- R25: value 3.24k -> 5.05k; digikey 311-3.24KCRDKR-ND -> 13-RT0805BRD075K05LDKR-ND
Connections:
- net GND: now also R27.1
- net at R23.1, U11.6 (FB): now also JP6.2 (C); no longer R25.2
- new net R_fb_12: JP6.3 (B), R27.2
- new net R_fb_24: JP6.1 (A), R25.2
Other:
- moved on the sheet: R25

Commit message: incremental updates
Parts:
- C29, C40: digikey (none) -> 1276-2525-1-ND
- U10, U11: digikey (none) -> 5503-TPP60508L1-DF9R-SCT-ND
Changed lines of the file:
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@@
 			)
 		)
+		(property "digikey" "5503-TPP60508L1-DF9R-SCT-ND"
+			(at 193.04 132.08 0)
+			(effects
+				(font
+					(size 1.27 1.27)
+				)
+				(hide yes)
+			)
+		)
 		(pin "7"
 		)
@@
 			)
 		)
-		(property "digikey" ""
+		(property "digikey" "1276-2525-1-ND"
 			(at 184.15 151.13 0)
 			(effects
@@
 			)
 		)
-		(property "digikey" ""
+		(property "digikey" "1276-2525-1-ND"
 			(at 181.61 81.28 0)
 			(effects
@@
 			(effects
 				(font
+					(size 1.27 1.27)
+				)
+				(hide yes)
+			)
+		)
+		(property "digikey" "5503-TPP60508L1-DF9R-SCT-ND"
+			(at 190.5 62.23 0)
+			(effects
+				(font

Commit message: initial production
Parts:
- added TP4, TP5: TestPoint, TestPoint:TestPoint_Pad_D1.5mm, symbol Connector:TestPoint
- C22, C33: digikey (none) -> 478-KAF21KR72A104MUCT-ND
- C28, C39: digikey (none) -> 311-1107-1-ND
Connections:
- net 5v: now also TP4.1
- net Vreg2: now also TP5.1
Changed lines of the file:
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@@
 			)
 		)
-		(property "digikey" ""
+		(property "digikey" "478-KAF21KR72A104MUCT-ND"
 			(at 176.53 40.64 0)
 			(effects
@@
 	)
 	(symbol
+		(lib_id "Connector:TestPoint")
+		(at 270.51 120.65 0)
+		(unit 1)
+		(exclude_from_sim no)
+		(in_bom yes)
+		(on_board yes)
+		(dnp no)
+		(fields_autoplaced yes)
+		(property "Reference" "TP5"
+			(at 273.05 116.0779 0)
+			(effects
+				(font
+					(size 1.27 1.27)
+				)
+				(justify left)
+			)
+		)
+		(property "Value" "TestPoint"
+			(at 273.05 118.6179 0)
+			(effects
+				(font
+					(size 1.27 1.27)
+				)
+				(justify left)
+			)
+		)
+		(property "Footprint" "TestPoint:TestPoint_Pad_D1.5mm"
+			(at 275.59 120.65 0)
+			(effects
+				(font
+					(size 1.27 1.27)
+				)
+				(hide yes)
+			)
+		)
+		(property "Datasheet" "~"
+			(at 275.59 120.65 0)
+			(effects
+				(font
+					(size 1.27 1.27)
+				)
+				(hide yes)
+			)
+		)
+		(property "Description" "test point"
+			(at 270.51 120.65 0)
+			(effects
+				(font
+					(size 1.27 1.27)
+				)
+				(hide yes)
+			)
+		)
+		(pin "1"
+		)
+		(instances
+			(project ""
+				(path "/c80e2680-7312-4906-8194-724a8268cfde/0b5a332f-b32e-4359-8448-44e694f7fb70"
+					(reference "TP5")
+					(unit 1)
+				)
+			)
+		)
+	)
+	(symbol
 		(lib_id "Device:C")
 		(at 184.15 151.13 0)
@@
 			)
 		)
-		(property "digikey" ""
+		(property "digikey" "478-KAF21KR72A104MUCT-ND"
 			(at 179.07 109.22 0)
 			(effects
@@
 	)
 	(symbol
+		(lib_id "Connector:TestPoint")
+		(at 266.7 50.8 0)
+		(unit 1)
+		(exclude_from_sim no)
+		(in_bom yes)
+		(on_board yes)
+		(dnp no)
+		(fields_autoplaced yes)
+		(property "Reference" "TP4"
+			(at 269.24 46.2279 0)
+			(effects
+				(font
+					(size 1.27 1.27)
+				)
+				(justify left)
+			)
+		)
+		(property "Value" "TestPoint"
+			(at 269.24 48.7679 0)
+			(effects
+				(font
+					(size 1.27 1.27)
+				)
+				(justify left)
+			)
+		)
+		(property "Footprint" "TestPoint:TestPoint_Pad_D1.5mm"
+			(at 271.78 50.8 0)
+			(effects
+				(font
+					(size 1.27 1.27)
+				)
+				(hide yes)
+			)
+		)
+		(property "Datasheet" "~"
+			(at 271.78 50.8 0)
+			(effects
+				(font
+					(size 1.27 1.27)
+				)
+				(hide yes)
+			)
+		)
+		(property "Description" "test point"
+			(at 266.7 50.8 0)
+			(effects
+				(font
+					(size 1.27 1.27)
+				)
+				(hide yes)
+			)
+		)
+		(pin "1"
+		)
+		(instances
+			(project ""
+				(path "/c80e2680-7312-4906-8194-724a8268cfde/0b5a332f-b32e-4359-8448-44e694f7fb70"
+					(reference "TP4")
+					(unit 1)
+				)
+			)
+		)
+	)
+	(symbol
 		(lib_id "Device:L")
 		(at 229.87 50.8 90)
@@
 			)
 		)
-		(property "digikey" ""
+		(property "digikey" "311-1107-1-ND"
 			(at 194.31 77.47 0)
 			(effects
@@
 			)
 		)
-		(property "digikey" ""
+		(property "digikey" "311-1107-1-ND"
 			(at 196.85 147.32 0)
 			(effects

Commit message: v0.1 prototype definition
Parts:
- M10, M7, M8, M9: digikey (none) -> 36-24939CT-ND
- R27: digikey 13-RC0805FR-0710R5LDKR-ND -> 311-10.5KCRCT-ND
Changed lines of the file:
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@@
 			)
 		)
+		(property "digikey" "36-24939CT-ND"
+			(at 20.32 154.94 0)
+			(effects
+				(font
+					(size 1.27 1.27)
+				)
+				(hide yes)
+			)
+		)
 		(instances
 			(project "duet_pi"
@@
 			)
 		)
-		(property "digikey" "13-RC0805FR-0710R5LDKR-ND"
+		(property "digikey" "311-10.5KCRCT-ND"
 			(at 231.14 151.13 0)
 			(effects
@@
 			)
 		)
+		(property "digikey" "36-24939CT-ND"
+			(at 20.32 166.37 0)
+			(effects
+				(font
+					(size 1.27 1.27)
+				)
+				(hide yes)
+			)
+		)
 		(instances
 			(project "duet_pi"
@@
 			)
 		)
+		(property "digikey" "36-24939CT-ND"
+			(at 20.32 190.5 0)
+			(effects
+				(font
+					(size 1.27 1.27)
+				)
+				(hide yes)
+			)
+		)
 		(instances
 			(project "duet_pi"
@@
 			(at 20.32 180.34 0)
 			(effects
+				(font
+					(size 1.27 1.27)
+				)
+				(hide yes)
+			)
+		)
+		(property "digikey" "36-24939CT-ND"
+			(at 20.32 180.34 0)
+			(effects
