File: duet_pi/misc.kicad_sch (KiCad schematic)
At the start: 68 parts, among them J16 Screw_Terminal_01x10, J17 Conn_Coaxial, J18 Conn_02x13_Odd_Even, J19 Conn_02x13_Odd_Even, M10 M3 Solder Nut, M6 Fan, M7 M3 Solder Nut, M8 M3 Solder Nut, M9 M3 Solder Nut, U10 TPP60508, U11 TPP60508

Commit message: fix: 5A diodes in regulation stages
Parts:
- D4, D5: digikey 5399-SS310CT-ND -> 5399-SS510CT-ND
Changed lines of the file:
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@@
 			)
 		)
-		(property "digikey" "5399-SS310CT-ND "
+		(property "digikey" "5399-SS510CT-ND"
 			(at 226.06 133.35 90)
 			(effects
@@
 			)
 		)
-		(property "digikey" "5399-SS310CT-ND "
+		(property "digikey" "5399-SS510CT-ND"
 			(at 223.52 63.5 90)
 			(effects
