File: duet_pi/PCIe-M2.kicad_sch (KiCad schematic)
At the start: 25 parts, among them J15 Bus_M.2_Socket_M, M1 M.2 Solder Nut, M2 M.2 Solder Nut, M3 M.2 Solder Nut, M4 M.2 Solder Nut, M5 M.2 Screw, U8 ASEK-32.768KHZ-L-R-T, U9 AP3441SHE-7B

Commit message: add m.2 solder nut to BOM
Parts:
- M1, M2, M3, M4: digikey (none) -> 36-24929CT-ND
Changed lines of the file:
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@@
+			)
+		)
+		(property "digikey" "36-24929CT-ND"
+			(at 250.19 93.98 0)
+			(effects
+				(font
+					(size 1.27 1.27)
+				)
+				(hide yes)
 			)
 		)
@@
 			)
 		)
+		(property "digikey" "36-24929CT-ND"
+			(at 250.19 132.08 0)
+			(effects
+				(font
+					(size 1.27 1.27)
+				)
+				(hide yes)
+			)
+		)
 		(instances
 			(project "duet_pi"
@@
 			)
 		)
+		(property "digikey" "36-24929CT-ND"
+			(at 250.19 119.38 0)
+			(effects
+				(font
+					(size 1.27 1.27)
+				)
+				(hide yes)
+			)
+		)
 		(instances
 			(project "duet_pi"
@@
 			(at 250.19 106.68 0)
 			(effects
+				(font
+					(size 1.27 1.27)
+				)
+				(hide yes)
+			)
+		)
+		(property "digikey" "36-24929CT-ND"
+			(at 250.19 106.68 0)
+			(effects
