File: duet_pi/CM5_GPIO.kicad_sch (KiCad schematic)
At the start: 29 parts, among them J2 THD-20-R, J20 JST_SHBM04B-SRSS-TB, J3 THD-02-R, J4 THD-13-R, J5 Micro_SD_Card_Det, J6 Conn_01x03, J8 Conn_02x07_Odd_Even, SW1 Right angle Tact button, U1 TPD4EUSB30, U2 TPD4EUSB30, U3 MagJack-A70-112-331N126, U4 74LVC1G07SE-7, U5 RT9742GGJ5

Commit message: fix ethernet, fan header
Parts:
- J7: Field7 JST -> (none); Part Description 4 pin vertical 1mm pitch connector -> (none); digikey (none) -> WM4330-ND
- U3: digikey 535-14155-ND -> (none)
Changed lines of the file:
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@@
 			)
 		)
-		(property "digikey" "535-14155-ND"
-			(at 264.16 95.25 0)
-			(effects
-				(font
-					(size 1.27 1.27)
-				)
-				(hide yes)
-			)
-		)
 		(pin "1"
 		)
@@
 			)
 		)
-		(property "Description" ""
-			(at 168.91 177.8 0)
-			(effects
-				(font
-					(size 1.27 1.27)
-				)
-				(hide yes)
-			)
-		)
-		(property "Field4" ""
-			(at 168.91 177.8 0)
-			(effects
-				(font
-					(size 1.27 1.27)
-				)
-				(hide yes)
-			)
-		)
-		(property "Field5" ""
-			(at 168.91 177.8 0)
-			(effects
-				(font
-					(size 1.27 1.27)
-				)
-				(hide yes)
-			)
-		)
-		(property "Field6" ""
-			(at 168.91 177.8 0)
-			(effects
-				(font
-					(size 1.27 1.27)
-				)
-				(hide yes)
-			)
-		)
-		(property "Field7" "JST"
+		(property "Description" "4 pin fan header (molex kk254)"
 			(at 168.91 177.8 0)
 			(effects
@@
 			)
 		)
-		(property "Part Description" "4 pin vertical 1mm pitch connector"
+		(property "digikey" "WM4330-ND"
 			(at 168.91 177.8 0)
 			(effects

Commit message: fix pc fan header J7
Connections:
- net +5v: now also J7.2 (Pin_2); no longer J7.1 (Pin_1)
- net GND: now also J7.1 (Pin_1); no longer J7.3 (Pin_3)
- net at JP8.3 (B): now also J7.3 (Pin_3); no longer J7.4 (Pin_4)
- net at JP7.3 (B): now also J7.4 (Pin_4); no longer J7.2 (Pin_2)
Changed lines of the file:
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@@
 	(wire
 		(pts
+			(xy 161.29 177.8) (xy 163.83 177.8)
+		)
+		(stroke
+			(width 0)
+			(type default)
+		)
+	)
+	(wire
+		(pts
 			(xy 110.49 107.95) (xy 96.52 107.95)
 		)
@@
 	(wire
 		(pts
+			(xy 153.67 180.34) (xy 153.67 182.88)
+		)
+		(stroke
+			(width 0)
+			(type default)
+		)
+	)
+	(wire
+		(pts
 			(xy 185.42 95.25) (xy 196.85 95.25)
 		)
@@
 	(wire
 		(pts
+			(xy 156.21 182.88) (xy 163.83 182.88)
+		)
+		(stroke
+			(width 0)
+			(type default)
+		)
+	)
+	(wire
+		(pts
 			(xy 162.56 41.91) (xy 161.29 41.91)
 		)
@@
 	(wire
 		(pts
-			(xy 162.56 180.34) (xy 162.56 187.96)
-		)
-		(stroke
-			(width 0)
-			(type default)
-		)
-	)
-	(wire
-		(pts
 			(xy 20.32 54.61) (xy 35.56 54.61)
 		)
@@
 	(wire
 		(pts
+			(xy 153.67 180.34) (xy 163.83 180.34)
+		)
+		(stroke
+			(width 0)
+			(type default)
+		)
+	)
+	(wire
+		(pts
 			(xy 318.77 129.54) (xy 327.66 129.54)
 		)
@@
 	(wire
 		(pts
-			(xy 148.59 182.88) (xy 163.83 182.88)
-		)
-		(stroke
-			(width 0)
-			(type default)
-		)
-	)
-	(wire
-		(pts
 			(xy 96.52 52.07) (xy 97.79 52.07)
 		)
@@
 	(wire
 		(pts
-			(xy 161.29 175.26) (xy 163.83 175.26)
-		)
-		(stroke
-			(width 0)
-			(type solid)
-		)
-	)
-	(wire
-		(pts
 			(xy 137.16 69.85) (xy 148.59 69.85)
 		)
@@
 	(wire
 		(pts
+			(xy 153.67 182.88) (xy 148.59 182.88)
+		)
+		(stroke
+			(width 0)
+			(type default)
+		)
+	)
+	(wire
+		(pts
 			(xy 34.29 39.37) (xy 34.29 49.53)
 		)
@@
 	(wire
 		(pts
-			(xy 163.83 180.34) (xy 162.56 180.34)
-		)
-		(stroke
-			(width 0)
-			(type default)
-		)
-	)
-	(wire
-		(pts
 			(xy 20.32 34.29) (xy 35.56 34.29)
 		)
@@
 	(wire
 		(pts
-			(xy 148.59 177.8) (xy 163.83 177.8)
-		)
-		(stroke
-			(width 0)
-			(type default)
-		)
-	)
-	(wire
-		(pts
 			(xy 137.16 64.77) (xy 148.59 64.77)
 		)
@@
 	(wire
 		(pts
+			(xy 156.21 177.8) (xy 156.21 182.88)
+		)
+		(stroke
+			(width 0)
+			(type default)
+		)
+	)
+	(wire
+		(pts
 			(xy 228.6 125.73) (xy 214.63 125.73)
 		)
@@
 	(wire
 		(pts
+			(xy 160.02 170.18) (xy 160.02 172.72)
+		)
+		(stroke
+			(width 0)
+			(type default)
+		)
+	)
+	(wire
+		(pts
 			(xy 147.32 74.93) (xy 147.32 76.2)
 		)
@@
 	(wire
 		(pts
+			(xy 148.59 177.8) (xy 156.21 177.8)
+		)
+		(stroke
+			(width 0)
+			(type default)
+		)
+	)
+	(wire
+		(pts
 			(xy 17.78 182.88) (xy 17.78 185.42)
 		)
@@
 	(wire
 		(pts
+			(xy 163.83 170.18) (xy 160.02 170.18)
+		)
+		(stroke
+			(width 0)
+			(type default)
+		)
+	)
+	(wire
+		(pts
 			(xy 217.17 118.11) (xy 228.6 118.11)
 		)
@@
 		)
 	)
+	(wire
+		(pts
+			(xy 163.83 175.26) (xy 163.83 170.18)
+		)
+		(stroke
+			(width 0)
+			(type default)
+		)
+	)
 	(text "FAN connector\n"
 		(exclude_from_sim no)
-		(at 156.845 172.72 0)
+		(at 161.036 168.91 0)
 		(effects
 			(font
@@
 	(hierarchical_label "+5v"
 		(shape input)
-		(at 161.29 175.26 180)
+		(at 161.29 177.8 180)
 		(effects
 			(font
@@
 	(symbol
 		(lib_id "power:GND")
-		(at 162.56 187.96 0)
+		(at 160.02 172.72 0)
 		(unit 1)
 		(exclude_from_sim no)
@@
 		(dnp no)
 		(property "Reference" "#PWR020"
-			(at 162.56 194.31 0)
+			(at 160.02 179.07 0)
 			(effects
 				(font
@@
 		)
 		(property "Value" "GND"
-			(at 162.687 192.3542 0)
+			(at 156.718 174.498 0)
 			(effects
 				(font
@@
 		)
 		(property "Footprint" ""
-			(at 162.56 187.96 0)
+			(at 160.02 172.72 0)
 			(effects
 				(font
@@
 		)
 		(property "Datasheet" ""
-			(at 162.56 187.96 0)
+			(at 160.02 172.72 0)
 			(effects
 				(font
@@
 		)
 		(property "Description" "Power symbol creates a global label with name \"GND\" , ground"
-			(at 162.56 187.96 0)
+			(at 160.02 172.72 0)
 			(effects
 				(font
