File: duet_pi/duet_pi.kicad_pcb (KiCad board)
At the start: 4 copper layers, 134 x 140 mm, 128 parts, among them J1 USB_C_Receptacle_USB2.0, J10 690-019-298-412, J11 USB3_A, J12 THD-02-R, J13 Conn_01x22_Female, J14 WM1282DKR-ND, J15 Bus_M.2_Socket_M, J16 Screw_Terminal_01x10, J2 THD-20-R, J20 JST_SHBM04B-SRSS-TB, J3 THD-02-R, J4 THD-13-R, J5 Micro_SD_Card_Det, J6 Conn_01x03, J8 Conn_02x07_Odd_Even, J9 Conn_01x22_Female, M6 Fan, SW1 Right angle Tact button, U1 TPD4EUSB30, U10 TPP60508, U11 TPP60508, U2 TPD4EUSB30, U3 MagJack-A70-112-331N126, U4 74LVC1G07SE-7, U5 RT9742GGJ5, U6 RT9742SNGV, U7 AP22653W6, U8 ASEK-32.768KHZ-L-R-T, U9 AP3441SHE-7B

Commit message: fix pc fan header J7
Connections:
- J7 pad 1: /+5v -> GND
- J7 pad 2: Net-(J7-Pin_2) -> /+5v
- J7 pad 3: GND -> Net-(J7-Pin_3)
- JP7 pad 3: Net-(J7-Pin_2) -> Net-(J7-Pin_4)
- JP8 pad 3: Net-(J7-Pin_4) -> Net-(J7-Pin_3)
Routing:
- net /+5v: track 494.1 -> 476.9 mm, vias 14 -> 15
- net Net-(J7-Pin_2): track 7.62 -> 0.00 mm
- net Net-(J7-Pin_3): track 0.00 -> 4.32 mm
- net GND: track 399.7 -> 397.9 mm
Changed lines of the file:
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@@
 	(net 241 "/misc/R_fb_24")
 	(net 242 "/misc/R_fb_12")
-	(net 243 "Net-(J7-Pin_2)")
+	(net 243 "Net-(J7-Pin_3)")
 	(net 244 "Net-(J7-Pin_4)")
 	(net 245 "Net-(J20-Pin_2)")
@@
 			(layers "*.Cu" "*.Mask")
 			(remove_unused_layers no)
-			(net 2 "/+5v")
+			(net 1 "GND")
 			(pinfunction "Pin_1")
 			(pintype "passive")
@@
 			(layers "*.Cu" "*.Mask")
 			(remove_unused_layers no)
-			(net 243 "Net-(J7-Pin_2)")
+			(net 2 "/+5v")
 			(pinfunction "Pin_2")
 			(pintype "passive")
@@
 			(layers "*.Cu" "*.Mask")
 			(remove_unused_layers no)
-			(net 1 "GND")
+			(net 243 "Net-(J7-Pin_3)")
 			(pinfunction "Pin_3")
 			(pintype "passive")
@@
 			(size 1 0.5)
 			(layers "B.Cu" "B.Mask")
-			(net 244 "Net-(J7-Pin_4)")
+			(net 243 "Net-(J7-Pin_3)")
 			(pinfunction "B")
 			(pintype "passive")
@@
 			(size 1 0.5)
 			(layers "B.Cu" "B.Mask")
-			(net 243 "Net-(J7-Pin_2)")
+			(net 244 "Net-(J7-Pin_4)")
 			(pinfunction "B")
 			(pintype "passive")
@@
 	)
 	(segment
-		(start 66.4 93.45)
-		(end 64.59 93.45)
-		(width 1)
-		(layer "In1.Cu")
-		(net 1)
-	)
-	(segment
 		(start 43.7 99.24)
 		(end 43.72 99.26)
@@
 	)
 	(segment
-		(start 70.06 103.52)
-		(end 71.22 102.36)
-		(width 0.13)
+		(start 67.885 103.52)
+		(end 70.11 105.745)
+		(width 0.3)
 		(layer "F.Cu")
 		(net 2)
@@
 	)
 	(segment
-		(start 71.22 93.19)
-		(end 66.4 88.37)
-		(width 0.13)
+		(start 151.5 110.3)
+		(end 151.5 123.92)
+		(width 0.5)
 		(layer "F.Cu")
 		(net 2)
 	)
 	(segment
-		(start 151.5 110.3)
-		(end 151.5 123.92)
-		(width 0.5)
+		(start 70.11 105.745)
+		(end 70.11 105.985537)
+		(width 0.3)
 		(layer "F.Cu")
 		(net 2)
@@
 	)
 	(segment
-		(start 67.885 103.52)
-		(end 70.06 103.52)
-		(width 0.13)
-		(layer "F.Cu")
-		(net 2)
-	)
-	(segment
-		(start 71.22 102.36)
-		(end 71.22 93.19)
-		(width 0.13)
-		(layer "F.Cu")
-		(net 2)
-	)
-	(segment
 		(start 141.54 104.97)
 		(end 141.54 104.63)
@@
 		(net 2)
 	)
+	(via
+		(at 70.11 105.985537)
+		(size 0.6)
+		(drill 0.3)
+		(layers "F.Cu" "B.Cu")
+		(net 2)
+	)
 	(segment
 		(start 69.03 154.08)
@@
 	)
 	(segment
-		(start 71.9 88.86)
-		(end 71.9 104.195537)
-		(width 3.5)
-		(layer "B.Cu")
-		(net 2)
-	)
-	(segment
 		(start 70.11 105.985537)
 		(end 70.11 118.56)
@@
 	)
 	(segment
-		(start 71.41 88.37)
-		(end 71.9 88.86)
-		(width 2)
-		(layer "B.Cu")
-		(net 2)
-	)
-	(segment
-		(start 71.86 88.82)
-		(end 71.9 88.86)
-		(width 1)
+		(start 71.9 90.8)
+		(end 71.9 104.195537)
+		(width 3.5)
 		(layer "B.Cu")
 		(net 2)
@@
 	)
 	(segment
-		(start 66.4 88.37)
-		(end 71.41 88.37)
-		(width 2)
-		(layer "B.Cu")
-		(net 2)
-	)
-	(segment
-		(start 66.4 88.37)
-		(end 54.37 88.37)
-		(width 2)
-		(layer "B.Cu")
-		(net 2)
-	)
-	(segment
 		(start 72.075 151.035)
 		(end 72.465 151.035)
@@
 	)
 	(segment
+		(start 66.4 90.91)
+		(end 71.79 90.91)
+		(width 2)
+		(layer "B.Cu")
+		(net 2)
+	)
+	(segment
 		(start 73.95 69.63)
 		(end 113.2 69.63)
@@
 	)
 	(segment
+		(start 67.062983 90.729688)
+		(end 66.580312 90.729688)
+		(width 0.13)
+		(layer "B.Cu")
+		(net 2)
+	)
+	(segment
+		(start 71.79 90.91)
+		(end 71.9 90.8)
+		(width 2)
+		(layer "B.Cu")
+		(net 2)
+	)
+	(segment
+		(start 71.9 88.86)
+		(end 71.9 90.8)
+		(width 3.5)
+		(layer "B.Cu")
+		(net 2)
+	)
+	(segment
 		(start 113.915 88.695)
 		(end 120.75 95.53)
@@
 	)
 	(segment
-		(start 54.37 88.37)
-		(end 44.18 98.56)
-		(width 2)
-		(layer "B.Cu")
-		(net 2)
-	)
-	(segment
 		(start 140.51 104.825)
 		(end 140.995 104.825)
@@
 	)
 	(segment
+		(start 66.4 90.91)
+		(end 51.83 90.91)
+		(width 2)
+		(layer "B.Cu")
+		(net 2)
+	)
+	(segment
+		(start 51.83 90.91)
+		(end 44.18 98.56)
+		(width 2)
+		(layer "B.Cu")
+		(net 2)
+	)
+	(segment
 		(start 140.995 104.825)
 		(end 141.34 105.17)
@@
 	)
 	(segment
-		(start 69.425 93.091705)
-		(end 67.062983 90.729688)
-		(width 0.13)
-		(layer "B.Cu")
-		(net 243)
-	)
-	(segment
-		(start 67.062983 90.729688)
-		(end 66.580312 90.729688)
-		(width 0.13)
+		(start 63.92 95.93)
+		(end 66.4 93.45)
+		(width 0.3)
 		(layer "B.Cu")
 		(net 243)
 	)
 	(segment
-		(start 69.425 95.735)
-		(end 69.425 93.091705)
-		(width 0.13)
+		(start 63.92 96.74)
+		(end 63.92 95.93)
+		(width 0.3)
 		(layer "B.Cu")
 		(net 243)
@@
 	(segment
 		(start 68.61 96.55)
-		(end 69.425 95.735)
-		(width 0.13)
-		(layer "B.Cu")
-		(net 243)
-	)
-	(segment
-		(start 64.99 95.89)
-		(end 65.09 95.99)
-		(width 0.13)
-		(layer "B.Cu")
-		(net 244)
-	)
-	(segment
-		(start 64.77 95.89)
-		(end 64.99 95.89)
-		(width 0.13)
-		(layer "B.Cu")
-		(net 244)
-	)
-	(segment
-		(start 63.92 96.74)
-		(end 64.77 95.89)
-		(width 0.13)
+		(end 66.96 96.55)
+		(width 0.3)
 		(layer "B.Cu")
 		(net 244)
 	)
 	(segment
-		(start 65.09 95.99)
+		(start 66.96 96.55)
 		(end 66.4 95.99)
-		(width 0.13)
+		(width 0.3)
 		(layer "B.Cu")
 		(net 244)
